Commit message: 03.23. v6 sim2real tuning complete

File: source/FABRICS/src/fabrics_sim/models/robots/urdf/openarm_tesollo/openarm_tesollo.urdf (robot description, URDF)
Before this commit: robot open_tesollo, 57 links, 56 joints
Links:
- added link rl_dg_1_tip
- added link rl_dg_2_tip
- added link rl_dg_3_tip
- added link rl_dg_4_tip
- added link rl_dg_5_tip
Joints:
- added joint rl_dg_1_tip_joint: type fixed, parent tesollo_right_rl_dg_1_4, child rl_dg_1_tip, origin xyz=0. 0.0363 0. rpy=0. 0. 0.
- added joint rl_dg_2_tip_joint: type fixed, parent tesollo_right_rl_dg_2_4, child rl_dg_2_tip, origin xyz=0. 0. 0.0255 rpy=0. 0. 0.
- added joint rl_dg_3_tip_joint: type fixed, parent tesollo_right_rl_dg_3_4, child rl_dg_3_tip, origin xyz=0. 0. 0.0255 rpy=0. 0. 0.
- added joint rl_dg_4_tip_joint: type fixed, parent tesollo_right_rl_dg_4_4, child rl_dg_4_tip, origin xyz=0. 0. 0.0255 rpy=0. 0. 0.
- added joint rl_dg_5_tip_joint: type fixed, parent tesollo_right_rl_dg_5_4, child rl_dg_5_tip, origin xyz=0. 0. 0.0363 rpy=0. 0. 0.
