Commit message: feat(fabrics): fabric URDF 3종을 DG-5FS(bi_s_rl) 기구학으로 갱신 [P0]
로봇 자산이 openarm_tesollo_bi_rl(DG-5F) → openarm_tesollo_bi_s_rl(DG-5FS)로
바뀌었다. 조인트/링크 이름은 동일하지만 기구학이 전면 재정의됐다:
  회전축     0 1 0 / 1 0 0 → 0 0 1 (전부, origin rpy 도입)
  마디 길이  PIP/DIP 0.0388 → 0.0334 m (14% 단축), tip 0.0255 → 0.018
  palm 오프셋 0.0698 → 0.015 m
  조인트 한계 20개 중 10개 변경 (엄지 _1: ±0.38/0.89 → ±1.571)

Fabrics 는 자산과 별개의 URDF 를 쓰고, 그 값이 구 DG-5F 와 완전히 일치했다.
갱신하지 않으면 palm pose IK 가 존재하지 않는 손을 푼다.

★부수 발견: 자산 재생성으로 mount 도 0.0595695 → 0.0495 (−10.07mm) 바뀌었다.
  fabric 은 구 mount 로 접혀 있어 **DG-5FS 전환과 무관하게 이미 10mm 어긋난 상태**였다.
  따라서 palm 오프셋 변화분만 옮기는 델타 방식은 틀리고, 손목→palm 체인을
  자산에서 절대 재계산해야 한다(0.1333695 → 0.0685).

변경:
- openarm_tesollo / _left / _sensor 3종의 손 revolute 20개(origin·axis·limit),
  palm_link_joint, tip 고정조인트 갱신
- 생성기 scripts/tools/gen_fabric_urdf_dg5fs.py 신설 (--verify 로 FK 대조)

검증: 무작위 관절각 5회 × 5손가락 = 25건 FK 대조
  갱신 전 최대 손끝 오차 29.251 mm → 갱신 후 0.000 mm (3종 모두)

미해결(다음 단계에서 검토):
- 충돌 구 프레임(tesollo_*_sphere2) 오프셋은 마디 단축 미반영. FK 정확도에는
  영향 없으나 충돌 근사가 헐거워진다.

File: source/FABRICS/src/fabrics_sim/models/robots/urdf/openarm_tesollo/openarm_tesollo.urdf (robot description, URDF)
Before this commit: robot open_tesollo, 62 links, 61 joints
Joints:
- joint palm_link_joint: origin xyz=0. 0.0000003 0.1333695 rpy=0. 0. -1.5707964 -> xyz=0 3e-07 0.0685 rpy=0. 0. -1.5707964
- joint rj_dg_1_1: axis 1. 0. 0. -> 0 0 1; limit lower=-0.3839724 upper=0.8901179 effort=7.5 velocity=3.1415927 -> lower=-1.5707963267948966 upper=1.5707963267948966 effort=7.5 velocity=3.1415927; origin xyz=-0.0162 0.019 0.0128 rpy=0. 0. 0. -> xyz=0.0017 0.018 0.0298 rpy=1.5708 0 1.5708
- joint rj_dg_1_2: axis 0. 0. 1. -> 0 0 1; limit lower=-3.1415927 upper=0. effort=7.5 velocity=3.1415927 -> lower=-2.670353755551324 upper=0 effort=7.5 velocity=3.1415927; origin xyz=0.04195 0. 0.  rpy=0. 0. 0. -> xyz=0 0 0.0262 rpy=-1.5708 0 0
- joint rj_dg_1_3: axis 1. 0. 0. -> 0 0 1; limit lower=-1.5707963 upper=1.5707963 effort=7.5 velocity=3.1415927 -> lower=-1.5707963267948966 upper=1.5707963267948966 effort=7.5 velocity=3.1415927; origin xyz=0. 0.031 0.  rpy=0. 0. 0. -> xyz=0.0381 0 0 rpy=1.5708 0 0
- joint rj_dg_1_4: axis 1. 0. 0. -> 0 0 1; limit lower=-1.5707963 upper=1.5707963 effort=7.5 velocity=3.1415927 -> lower=-1.5707963267948966 upper=1.5707963267948966 effort=7.5 velocity=3.1415927; origin xyz=0. 0.0388 0.  rpy=0. 0. 0. -> xyz=0.0334 0 0 rpy=0 0 0
- joint rj_dg_2_1: axis 1. 0. 0. -> 0 0 1; limit lower=-0.418879 upper=0.6108652 effort=7.5 velocity=3.1415927 -> lower=-0.8377580409572782 upper=0.2617993877991494 effort=7.5 velocity=3.1415927; origin xyz=-0.0071 0.027 0.0661 rpy=0. 0. 0. -> xyz=0.0017 0.028 0.08365 rpy=3.1416 -1.5708 0
- joint rj_dg_2_2: axis 0. 1. 0. -> 0 0 -1; limit lower=0. upper=2.0071286 effort=7.5 velocity=3.1415927 -> lower=0 upper=2.199114857512855 effort=7.5 velocity=3.1415927; origin xyz=0.01765 0. 0.0265  rpy=0. 0. 0. -> xyz=0.02415 0 0.0126 rpy=-1.5708 0 0
- joint rj_dg_2_3: axis 0. 1. 0. -> 0 0 1; limit lower=-1.5707963 upper=1.5707963 effort=7.5 velocity=3.1415927 -> lower=-1.5707963267948966 upper=1.5707963267948966 effort=7.5 velocity=3.1415927; origin xyz=0. 0. 0.0388 rpy=0. 0. 0. -> xyz=0.0334 0 0 rpy=3.1416 0 0
- joint rj_dg_2_4: axis 0. 1. 0. -> 0 0 1; limit lower=-1.5707963 upper=1.5707963 effort=7.5 velocity=3.1415927 -> lower=-1.5707963267948966 upper=1.5707963267948966 effort=7.5 velocity=3.1415927; origin xyz=0. 0. 0.0388 rpy=0. 0. 0. -> xyz=0.0334 0 0 rpy=0 0 0
- joint rj_dg_3_1: axis 1. 0. 0. -> 0 0 1; limit lower=-0.6108652 upper=0.6108652 effort=7.5 velocity=3.1415927 -> lower=-0.5759586531581288 upper=0.7330382858376184 effort=7.5 velocity=3.1415927; origin xyz=-0.0071 0.0025 0.0701 rpy=0. 0. 0. -> xyz=0.0017 0.005 0.08865 rpy=3.1416 -1.5708 0
- joint rj_dg_3_2: axis 0. 1. 0. -> 0 0 -1; limit lower=0. upper=1.9547686 effort=7.5 velocity=3.1415927 -> lower=0 upper=2.2689280275926285 effort=7.5 velocity=3.1415927; origin xyz=0.01765 0. 0.0265  rpy=0. 0. 0. -> xyz=0.02415 0 0.0126 rpy=-1.5708 0 0
- joint rj_dg_3_3: axis 0. 1. 0. -> 0 0 1; limit lower=-1.5707963 upper=1.5707963 effort=7.5 velocity=3.1415927 -> lower=-1.5707963267948966 upper=1.5707963267948966 effort=7.5 velocity=3.1415927; origin xyz=0. 0. 0.0388 rpy=0. 0. 0. -> xyz=0.0334 0 0 rpy=3.1416 0 0
- joint rj_dg_3_4: axis 0. 1. 0. -> 0 0 1; limit lower=-1.5707963 upper=1.5707963 effort=7.5 velocity=3.1415927 -> lower=-1.5707963267948966 upper=1.5707963267948966 effort=7.5 velocity=3.1415927; origin xyz=0. 0. 0.0388 rpy=0. 0. 0. -> xyz=0.0334 0 0 rpy=0 0 0
- joint rj_dg_4_1: axis 1. 0. 0. -> 0 0 1; limit lower=-0.6108652 upper=0.418879 effort=7.5 velocity=3.1415927 -> lower=-0.20943951023931956 upper=0.8377580409572782 effort=7.5 velocity=3.1415927; origin xyz=-0.0071 -0.022 0.0621 rpy=0. 0. 0. -> xyz=0.0013 -0.018 0.08065 rpy=3.1416 -1.5708 0
- joint rj_dg_4_2: axis 0. 1. 0. -> 0 0 -1; limit lower=0. upper=1.9024088 effort=7.5 velocity=3.1415927 -> lower=0 upper=2.2165681500327987 effort=7.5 velocity=3.1415927; origin xyz=0.01765 0. 0.0265  rpy=0. 0. 0. -> xyz=0.02415 0 0.0126 rpy=-1.5708 0 0
- joint rj_dg_4_3: axis 0. 1. 0. -> 0 0 1; limit lower=-1.5707963 upper=1.5707963 effort=7.5 velocity=3.1415927 -> lower=-1.5707963267948966 upper=1.5707963267948966 effort=7.5 velocity=3.1415927; origin xyz=0. 0. 0.0388 rpy=0. 0. 0. -> xyz=0.0334 0 0 rpy=3.1416 0 0
- joint rj_dg_4_4: axis 0. 1. 0. -> 0 0 1; limit lower=-1.5707963 upper=1.5707963 effort=7.5 velocity=3.1415927 -> lower=-1.5707963267948966 upper=1.5707963267948966 effort=7.5 velocity=3.1415927; origin xyz=0. 0. 0.0388 rpy=0. 0. 0. -> xyz=0.0334 0 0 rpy=0 0 0
- joint rj_dg_5_1: axis 0. 0. 1. -> 0 0 1; limit lower=-0.0174533 upper=1.0471976 effort=7.5 velocity=3.1415927 -> lower=0 upper=1.0471975511965976 effort=7.5 velocity=3.1415927; origin xyz=0.0103 -0.0195 0.0182 rpy=0. 0. 0. -> xyz=0.013 -0.01805 0.0364 rpy=0 0 -1.5708
- joint rj_dg_5_2: axis 1. 0. 0. -> 0 0 1; limit lower=-0.418879 upper=0.6108652 effort=7.5 velocity=3.1415927 -> lower=-0.6457718232379019 upper=1.5707963267948966 effort=7.5 velocity=3.1415927; origin xyz=0. -0.028 0.0381 rpy=0. 0. 0. -> xyz=0.02445 0 0.0307 rpy=-1.5708 0 0
- joint rj_dg_5_3: axis 0. 1. 0. -> 0 0 1; limit lower=-1.5707963 upper=1.5707963 effort=7.5 velocity=3.1415927 -> lower=-1.5707963267948966 upper=1.5707963267948966 effort=7.5 velocity=3.1415927; origin xyz=0. 0. 0.031 rpy=0. 0. 0. -> xyz=0 -0.0272 0 rpy=1.5708 0 -1.5708
- joint rj_dg_5_4: axis 0. 1. 0. -> 0 0 1; limit lower=-1.5707963 upper=1.5707963 effort=7.5 velocity=3.1415927 -> lower=-1.5707963267948966 upper=1.5707963267948966 effort=7.5 velocity=3.1415927; origin xyz=0. 0. 0.0388 rpy=0. 0. 0. -> xyz=0.0334 0 0 rpy=0 0 0
- joint rl_dg_1_tip_joint: origin xyz=0. 0.0363 0. rpy=0. 0. 0. -> xyz=0.0289 0 0 rpy=0 0 0
- joint rl_dg_2_tip_joint: origin xyz=0. 0. 0.0255 rpy=0. 0. 0. -> xyz=0.018 0 0 rpy=0 0 0
- joint rl_dg_3_tip_joint: origin xyz=0. 0. 0.0255 rpy=0. 0. 0. -> xyz=0.018 0 0 rpy=0 0 0
- joint rl_dg_4_tip_joint: origin xyz=0. 0. 0.0255 rpy=0. 0. 0. -> xyz=0.018 0 0 rpy=0 0 0
- joint rl_dg_5_tip_joint: origin xyz=0. 0. 0.0363 rpy=0. 0. 0. -> xyz=0.0289 0 0 rpy=0 0 0

File: source/FABRICS/src/fabrics_sim/models/robots/urdf/openarm_tesollo_left/openarm_tesollo_left.urdf (robot description, URDF)
Before this commit: robot openarm_tesollo_left, 62 links, 61 joints
Joints:
- joint palm_link_joint: origin xyz=0 -3e-07 0.1333695 rpy=0 0 1.5707964 -> xyz=0 -3e-07 0.0685 rpy=0 0 1.5707964
- joint rj_dg_1_1: axis 1 0 0 -> 0 0 1; limit lower=-0.8901179 upper=0.3839724 effort=7.5 velocity=3.1415927 -> lower=-1.5707963267948966 upper=1.5707963267948966 effort=7.5 velocity=3.1415927; origin xyz=-0.0162 -0.019 0.0128 rpy=0 0 0 -> xyz=0.0017 -0.018 0.0298 rpy=-1.5708 0 -1.5708
- joint rj_dg_1_2: limit lower=-0 upper=3.1415927 effort=7.5 velocity=3.1415927 -> lower=0 upper=2.670353755551324 effort=7.5 velocity=3.1415927; origin xyz=0.04195 0 0 rpy=0 0 0 -> xyz=0 0 0.0262 rpy=1.5708 0 0
- joint rj_dg_1_3: axis 1 0 0 -> 0 0 1; limit lower=-1.5707963 upper=1.5707963 effort=7.5 velocity=3.1415927 -> lower=-1.5707963267948966 upper=1.5707963267948966 effort=7.5 velocity=3.1415927; origin xyz=0 -0.031 0 rpy=0 0 0 -> xyz=0.0381 0 0 rpy=-1.5708 0 0
- joint rj_dg_1_4: axis 1 0 0 -> 0 0 1; limit lower=-1.5707963 upper=1.5707963 effort=7.5 velocity=3.1415927 -> lower=-1.5707963267948966 upper=1.5707963267948966 effort=7.5 velocity=3.1415927; origin xyz=0 -0.0388 0 rpy=0 0 0 -> xyz=0.0334 0 0 rpy=0 0 0
- joint rj_dg_2_1: axis 1 0 0 -> 0 0 1; limit lower=-0.6108652 upper=0.418879 effort=7.5 velocity=3.1415927 -> lower=-0.2617993877991494 upper=0.8377580409572782 effort=7.5 velocity=3.1415927; origin xyz=-0.0071 -0.027 0.0661 rpy=0 0 0 -> xyz=0.0017 -0.028 0.08365 rpy=3.1416 -1.5708 0
- joint rj_dg_2_2: axis 0 1 0 -> 0 0 1; limit lower=0 upper=2.0071286 effort=7.5 velocity=3.1415927 -> lower=0 upper=2.199114857512855 effort=7.5 velocity=3.1415927; origin xyz=0.01765 0 0.0265 rpy=0 0 0 -> xyz=0.02415 0 0.0126 rpy=1.5708 0 0
- joint rj_dg_2_3: axis 0 1 0 -> 0 0 1; limit lower=-1.5707963 upper=1.5707963 effort=7.5 velocity=3.1415927 -> lower=-1.5707963267948966 upper=1.5707963267948966 effort=7.5 velocity=3.1415927; origin xyz=0 0 0.0388 rpy=0 0 0 -> xyz=0.0334 0 0 rpy=0 0 0
- joint rj_dg_2_4: axis 0 1 0 -> 0 0 1; limit lower=-1.5707963 upper=1.5707963 effort=7.5 velocity=3.1415927 -> lower=-1.5707963267948966 upper=1.5707963267948966 effort=7.5 velocity=3.1415927; origin xyz=0 0 0.0388 rpy=0 0 0 -> xyz=0.0334 0 0 rpy=0 0 0
- joint rj_dg_3_1: axis 1 0 0 -> 0 0 1; limit lower=-0.6108652 upper=0.6108652 effort=7.5 velocity=3.1415927 -> lower=-0.7330382858376184 upper=0.5759586531581288 effort=7.5 velocity=3.1415927; origin xyz=-0.0071 -0.0025 0.0701 rpy=0 0 0 -> xyz=0.0017 -0.005 0.08865 rpy=3.1416 -1.5708 0
- joint rj_dg_3_2: axis 0 1 0 -> 0 0 1; limit lower=0 upper=1.9547686 effort=7.5 velocity=3.1415927 -> lower=0 upper=2.2689280275926285 effort=7.5 velocity=3.1415927; origin xyz=0.01765 0 0.0265 rpy=0 0 0 -> xyz=0.02415 0 0.0126 rpy=1.5708 0 0
- joint rj_dg_3_3: axis 0 1 0 -> 0 0 1; limit lower=-1.5707963 upper=1.5707963 effort=7.5 velocity=3.1415927 -> lower=-1.5707963267948966 upper=1.5707963267948966 effort=7.5 velocity=3.1415927; origin xyz=0 0 0.0388 rpy=0 0 0 -> xyz=0.0334 0 0 rpy=0 0 0
- joint rj_dg_3_4: axis 0 1 0 -> 0 0 1; limit lower=-1.5707963 upper=1.5707963 effort=7.5 velocity=3.1415927 -> lower=-1.5707963267948966 upper=1.5707963267948966 effort=7.5 velocity=3.1415927; origin xyz=0 0 0.0388 rpy=0 0 0 -> xyz=0.0334 0 0 rpy=0 0 0
- joint rj_dg_4_1: axis 1 0 0 -> 0 0 1; limit lower=-0.418879 upper=0.6108652 effort=7.5 velocity=3.1415927 -> lower=-0.8377580409572782 upper=0.20943951023931956 effort=7.5 velocity=3.1415927; origin xyz=-0.0071 0.022 0.0621 rpy=0 0 0 -> xyz=0.0017 0.018 0.08065 rpy=3.1416 -1.5708 0
- joint rj_dg_4_2: axis 0 1 0 -> 0 0 1; limit lower=0 upper=1.9024088 effort=7.5 velocity=3.1415927 -> lower=0 upper=2.2165681500327987 effort=7.5 velocity=3.1415927; origin xyz=0.01765 0 0.0265 rpy=0 0 0 -> xyz=0.02415 0 0.0126 rpy=1.5708 0 0
- joint rj_dg_4_3: axis 0 1 0 -> 0 0 1; limit lower=-1.5707963 upper=1.5707963 effort=7.5 velocity=3.1415927 -> lower=-1.5707963267948966 upper=1.5707963267948966 effort=7.5 velocity=3.1415927; origin xyz=0 0 0.0388 rpy=0 0 0 -> xyz=0.0334 0 0 rpy=0 0 0
- joint rj_dg_4_4: axis 0 1 0 -> 0 0 1; limit lower=-1.5707963 upper=1.5707963 effort=7.5 velocity=3.1415927 -> lower=-1.5707963267948966 upper=1.5707963267948966 effort=7.5 velocity=3.1415927; origin xyz=0 0 0.0388 rpy=0 0 0 -> xyz=0.0334 0 0 rpy=0 0 0
- joint rj_dg_5_1: limit lower=-1.0471976 upper=0.0174533 effort=7.5 velocity=3.1415927 -> lower=-1.0471975511965976 upper=0 effort=7.5 velocity=3.1415927; origin xyz=0.0103 0.0195 0.0182 rpy=0 0 0 -> xyz=0.013 0.01805 0.0364 rpy=0 0 1.5708
- joint rj_dg_5_2: axis 1 0 0 -> 0 0 1; limit lower=-0.6108652 upper=0.418879 effort=7.5 velocity=3.1415927 -> lower=-1.5707963267948966 upper=0.6457718232379019 effort=7.5 velocity=3.1415927; origin xyz=0 0.028 0.0381 rpy=0 0 0 -> xyz=0.02445 0 0.0307 rpy=1.5708 0 0
- joint rj_dg_5_3: axis 0 1 0 -> 0 0 1; limit lower=-1.5707963 upper=1.5707963 effort=7.5 velocity=3.1415927 -> lower=-1.5707963267948966 upper=1.5707963267948966 effort=7.5 velocity=3.1415927; origin xyz=0 0 0.031 rpy=0 0 0 -> xyz=0 0.0272 0 rpy=1.5708 0 1.5708
- joint rj_dg_5_4: axis 0 1 0 -> 0 0 1; limit lower=-1.5707963 upper=1.5707963 effort=7.5 velocity=3.1415927 -> lower=-1.5707963267948966 upper=1.5707963267948966 effort=7.5 velocity=3.1415927; origin xyz=0 0 0.0388 rpy=0 0 0 -> xyz=0.0334 0 0 rpy=0 0 0
- joint rl_dg_1_tip_joint: origin xyz=0 -0.0363 0 rpy=0 0 0 -> xyz=0.0289 0 0 rpy=0 0 0
- joint rl_dg_2_tip_joint: origin xyz=0 0 0.0255 rpy=0 0 0 -> xyz=0.018 0 0 rpy=0 0 0
- joint rl_dg_3_tip_joint: origin xyz=0 0 0.0255 rpy=0 0 0 -> xyz=0.018 0 0 rpy=0 0 0
- joint rl_dg_4_tip_joint: origin xyz=0 0 0.0255 rpy=0 0 0 -> xyz=0.018 0 0 rpy=0 0 0
- joint rl_dg_5_tip_joint: origin xyz=0 0 0.0363 rpy=0 0 0 -> xyz=0.0289 0 0 rpy=0 0 0

File: source/FABRICS/src/fabrics_sim/models/robots/urdf/openarm_tesollo_sensor/openarm_tesollo_sensor.urdf (robot description, URDF)
Before this commit: robot openarm_tesollo_sensor, 63 links, 62 joints
Joints:
- joint palm_link_joint: origin xyz=0. 0.0000003 0.1333695 rpy=0. 0. -1.5707964 -> xyz=0 3e-07 0.0685 rpy=0. 0. -1.5707964
- joint rj_dg_1_1: axis 1. 0. 0. -> 0 0 1; limit lower=-0.3839724 upper=0.8901179 effort=7.5 velocity=3.1415927 -> lower=-1.5707963267948966 upper=1.5707963267948966 effort=7.5 velocity=3.1415927; origin xyz=-0.0162 0.019 0.0128 rpy=0. 0. 0. -> xyz=0.0017 0.018 0.0298 rpy=1.5708 0 1.5708
- joint rj_dg_1_2: axis 0. 0. 1. -> 0 0 1; limit lower=-3.1415927 upper=0. effort=7.5 velocity=3.1415927 -> lower=-2.670353755551324 upper=0 effort=7.5 velocity=3.1415927; origin xyz=0.04195 0. 0.  rpy=0. 0. 0. -> xyz=0 0 0.0262 rpy=-1.5708 0 0
- joint rj_dg_1_3: axis 1. 0. 0. -> 0 0 1; limit lower=-1.5707963 upper=1.5707963 effort=7.5 velocity=3.1415927 -> lower=-1.5707963267948966 upper=1.5707963267948966 effort=7.5 velocity=3.1415927; origin xyz=0. 0.031 0.  rpy=0. 0. 0. -> xyz=0.0381 0 0 rpy=1.5708 0 0
- joint rj_dg_1_4: axis 1. 0. 0. -> 0 0 1; limit lower=-1.5707963 upper=1.5707963 effort=7.5 velocity=3.1415927 -> lower=-1.5707963267948966 upper=1.5707963267948966 effort=7.5 velocity=3.1415927; origin xyz=0. 0.0388 0.  rpy=0. 0. 0. -> xyz=0.0334 0 0 rpy=0 0 0
- joint rj_dg_1_tip: origin xyz=0. 0.0363 0. rpy=0. 0. 0. -> xyz=0.0289 0 0 rpy=0 0 0
- joint rj_dg_2_1: axis 1. 0. 0. -> 0 0 1; limit lower=-0.418879 upper=0.6108652 effort=7.5 velocity=3.1415927 -> lower=-0.8377580409572782 upper=0.2617993877991494 effort=7.5 velocity=3.1415927; origin xyz=-0.0071 0.027 0.0661 rpy=0. 0. 0. -> xyz=0.0017 0.028 0.08365 rpy=3.1416 -1.5708 0
- joint rj_dg_2_2: axis 0. 1. 0. -> 0 0 -1; limit lower=0. upper=2.0071286 effort=7.5 velocity=3.1415927 -> lower=0 upper=2.199114857512855 effort=7.5 velocity=3.1415927; origin xyz=0.01765 0. 0.0265  rpy=0. 0. 0. -> xyz=0.02415 0 0.0126 rpy=-1.5708 0 0
- joint rj_dg_2_3: axis 0. 1. 0. -> 0 0 1; limit lower=-1.5707963 upper=1.5707963 effort=7.5 velocity=3.1415927 -> lower=-1.5707963267948966 upper=1.5707963267948966 effort=7.5 velocity=3.1415927; origin xyz=0. 0. 0.0388 rpy=0. 0. 0. -> xyz=0.0334 0 0 rpy=3.1416 0 0
- joint rj_dg_2_4: axis 0. 1. 0. -> 0 0 1; limit lower=-1.5707963 upper=1.5707963 effort=7.5 velocity=3.1415927 -> lower=-1.5707963267948966 upper=1.5707963267948966 effort=7.5 velocity=3.1415927; origin xyz=0. 0. 0.0388 rpy=0. 0. 0. -> xyz=0.0334 0 0 rpy=0 0 0
- joint rj_dg_2_tip: origin xyz=0. 0. 0.0255 rpy=0. 0. 0. -> xyz=0.018 0 0 rpy=0 0 0
- joint rj_dg_3_1: axis 1. 0. 0. -> 0 0 1; limit lower=-0.6108652 upper=0.6108652 effort=7.5 velocity=3.1415927 -> lower=-0.5759586531581288 upper=0.7330382858376184 effort=7.5 velocity=3.1415927; origin xyz=-0.0071 0.0025 0.0701 rpy=0. 0. 0. -> xyz=0.0017 0.005 0.08865 rpy=3.1416 -1.5708 0
- joint rj_dg_3_2: axis 0. 1. 0. -> 0 0 -1; limit lower=0. upper=1.9547686 effort=7.5 velocity=3.1415927 -> lower=0 upper=2.2689280275926285 effort=7.5 velocity=3.1415927; origin xyz=0.01765 0. 0.0265  rpy=0. 0. 0. -> xyz=0.02415 0 0.0126 rpy=-1.5708 0 0
- joint rj_dg_3_3: axis 0. 1. 0. -> 0 0 1; limit lower=-1.5707963 upper=1.5707963 effort=7.5 velocity=3.1415927 -> lower=-1.5707963267948966 upper=1.5707963267948966 effort=7.5 velocity=3.1415927; origin xyz=0. 0. 0.0388 rpy=0. 0. 0. -> xyz=0.0334 0 0 rpy=3.1416 0 0
- joint rj_dg_3_4: axis 0. 1. 0. -> 0 0 1; limit lower=-1.5707963 upper=1.5707963 effort=7.5 velocity=3.1415927 -> lower=-1.5707963267948966 upper=1.5707963267948966 effort=7.5 velocity=3.1415927; origin xyz=0. 0. 0.0388 rpy=0. 0. 0. -> xyz=0.0334 0 0 rpy=0 0 0
- joint rj_dg_3_tip: origin xyz=0. 0. 0.0255 rpy=0. 0. 0. -> xyz=0.018 0 0 rpy=0 0 0
- joint rj_dg_4_1: axis 1. 0. 0. -> 0 0 1; limit lower=-0.6108652 upper=0.418879 effort=7.5 velocity=3.1415927 -> lower=-0.20943951023931956 upper=0.8377580409572782 effort=7.5 velocity=3.1415927; origin xyz=-0.0071 -0.022 0.0621 rpy=0. 0. 0. -> xyz=0.0013 -0.018 0.08065 rpy=3.1416 -1.5708 0
- joint rj_dg_4_2: axis 0. 1. 0. -> 0 0 -1; limit lower=0. upper=1.9024088 effort=7.5 velocity=3.1415927 -> lower=0 upper=2.2165681500327987 effort=7.5 velocity=3.1415927; origin xyz=0.01765 0. 0.0265  rpy=0. 0. 0. -> xyz=0.02415 0 0.0126 rpy=-1.5708 0 0
- joint rj_dg_4_3: axis 0. 1. 0. -> 0 0 1; limit lower=-1.5707963 upper=1.5707963 effort=7.5 velocity=3.1415927 -> lower=-1.5707963267948966 upper=1.5707963267948966 effort=7.5 velocity=3.1415927; origin xyz=0. 0. 0.0388 rpy=0. 0. 0. -> xyz=0.0334 0 0 rpy=3.1416 0 0
- joint rj_dg_4_4: axis 0. 1. 0. -> 0 0 1; limit lower=-1.5707963 upper=1.5707963 effort=7.5 velocity=3.1415927 -> lower=-1.5707963267948966 upper=1.5707963267948966 effort=7.5 velocity=3.1415927; origin xyz=0. 0. 0.0388 rpy=0. 0. 0. -> xyz=0.0334 0 0 rpy=0 0 0
- joint rj_dg_4_tip: origin xyz=0. 0. 0.0255 rpy=0. 0. 0. -> xyz=0.018 0 0 rpy=0 0 0
- joint rj_dg_5_1: axis 0. 0. 1. -> 0 0 1; limit lower=-0.0174533 upper=1.0471976 effort=7.5 velocity=3.1415927 -> lower=0 upper=1.0471975511965976 effort=7.5 velocity=3.1415927; origin xyz=0.0103 -0.0195 0.0182 rpy=0. 0. 0. -> xyz=0.013 -0.01805 0.0364 rpy=0 0 -1.5708
- joint rj_dg_5_2: axis 1. 0. 0. -> 0 0 1; limit lower=-0.418879 upper=0.6108652 effort=7.5 velocity=3.1415927 -> lower=-0.6457718232379019 upper=1.5707963267948966 effort=7.5 velocity=3.1415927; origin xyz=0. -0.028 0.0381 rpy=0. 0. 0. -> xyz=0.02445 0 0.0307 rpy=-1.5708 0 0
- joint rj_dg_5_3: axis 0. 1. 0. -> 0 0 1; limit lower=-1.5707963 upper=1.5707963 effort=7.5 velocity=3.1415927 -> lower=-1.5707963267948966 upper=1.5707963267948966 effort=7.5 velocity=3.1415927; origin xyz=0. 0. 0.031 rpy=0. 0. 0. -> xyz=0 -0.0272 0 rpy=1.5708 0 -1.5708
- joint rj_dg_5_4: axis 0. 1. 0. -> 0 0 1; limit lower=-1.5707963 upper=1.5707963 effort=7.5 velocity=3.1415927 -> lower=-1.5707963267948966 upper=1.5707963267948966 effort=7.5 velocity=3.1415927; origin xyz=0. 0. 0.0388 rpy=0. 0. 0. -> xyz=0.0334 0 0 rpy=0 0 0
- joint rj_dg_5_tip: origin xyz=0. 0. 0.0363 rpy=0. 0. 0. -> xyz=0.0289 0 0 rpy=0 0 0
