Commit message: refactor(fabrics): DG-5FS 전용 fabric URDF 분리 — 기존 URDF 원상 복구 [P0b]
사용자 지시: 기존 FABRICS 전용 URDF(구 DG-5F)는 그대로 두고 bi_s_rl 전용을 신설.
P0(95caa19)의 제자리 갱신을 되돌리고 전용 디렉토리로 재구성한다 — pour 등
구 자산 소비자를 보호하기 위함.

- openarm_tesollo / _left / _sensor URDF: 95caa19 이전 원본으로 복구
- 신설: models/robots/urdf/openarm_tesollo_bi_s/ (우), openarm_tesollo_bi_s_left/ (좌)
  · 원본 템플릿 복사 후 gen_fabric_urdf_dg5fs.py 적용, FK 대조 25건 오차 0.000mm
  · 우측 meshes 는 465MB 라 심볼릭 링크(../openarm_tesollo/meshes),
    좌측 URDF 는 원래 ../openarm_tesollo/meshes 상대참조라 링크 불필요
- OpenArmTeoslloLeftPoseFabric: robot_dir_name/robot_name 패스스루 추가(기본값 구 URDF)
- grasp 5개 태스크(main+reset fabric 10곳)에 bi_s(_left) 명시 배선

검증: 5개 태스크 전부 부팅 + 56관절 커버 + 20스텝 진행 OK
(obs 154/208/134/114/362D)

File: source/FABRICS/src/fabrics_sim/models/robots/urdf/openarm_tesollo_bi_s_left/openarm_tesollo_bi_s_left.urdf (robot description, URDF)
Before this commit: robot openarm_tesollo_left, 62 links, 61 joints
Joints:
- joint palm_link_joint: origin xyz=0 -3e-07 0.1333695 rpy=0 0 1.5707964 -> xyz=0 -3e-07 0.0685 rpy=0 0 1.5707964
- joint rj_dg_1_1: axis 1 0 0 -> 0 0 1; limit lower=-0.8901179 upper=0.3839724 effort=7.5 velocity=3.1415927 -> lower=-1.5707963267948966 upper=1.5707963267948966 effort=7.5 velocity=3.1415927; origin xyz=-0.0162 -0.019 0.0128 rpy=0 0 0 -> xyz=0.0017 -0.018 0.0298 rpy=-1.5708 0 -1.5708
- joint rj_dg_1_2: limit lower=-0 upper=3.1415927 effort=7.5 velocity=3.1415927 -> lower=0 upper=2.670353755551324 effort=7.5 velocity=3.1415927; origin xyz=0.04195 0 0 rpy=0 0 0 -> xyz=0 0 0.0262 rpy=1.5708 0 0
- joint rj_dg_1_3: axis 1 0 0 -> 0 0 1; limit lower=-1.5707963 upper=1.5707963 effort=7.5 velocity=3.1415927 -> lower=-1.5707963267948966 upper=1.5707963267948966 effort=7.5 velocity=3.1415927; origin xyz=0 -0.031 0 rpy=0 0 0 -> xyz=0.0381 0 0 rpy=-1.5708 0 0
- joint rj_dg_1_4: axis 1 0 0 -> 0 0 1; limit lower=-1.5707963 upper=1.5707963 effort=7.5 velocity=3.1415927 -> lower=-1.5707963267948966 upper=1.5707963267948966 effort=7.5 velocity=3.1415927; origin xyz=0 -0.0388 0 rpy=0 0 0 -> xyz=0.0334 0 0 rpy=0 0 0
- joint rj_dg_2_1: axis 1 0 0 -> 0 0 1; limit lower=-0.6108652 upper=0.418879 effort=7.5 velocity=3.1415927 -> lower=-0.2617993877991494 upper=0.8377580409572782 effort=7.5 velocity=3.1415927; origin xyz=-0.0071 -0.027 0.0661 rpy=0 0 0 -> xyz=0.0017 -0.028 0.08365 rpy=3.1416 -1.5708 0
- joint rj_dg_2_2: axis 0 1 0 -> 0 0 1; limit lower=0 upper=2.0071286 effort=7.5 velocity=3.1415927 -> lower=0 upper=2.199114857512855 effort=7.5 velocity=3.1415927; origin xyz=0.01765 0 0.0265 rpy=0 0 0 -> xyz=0.02415 0 0.0126 rpy=1.5708 0 0
- joint rj_dg_2_3: axis 0 1 0 -> 0 0 1; limit lower=-1.5707963 upper=1.5707963 effort=7.5 velocity=3.1415927 -> lower=-1.5707963267948966 upper=1.5707963267948966 effort=7.5 velocity=3.1415927; origin xyz=0 0 0.0388 rpy=0 0 0 -> xyz=0.0334 0 0 rpy=0 0 0
- joint rj_dg_2_4: axis 0 1 0 -> 0 0 1; limit lower=-1.5707963 upper=1.5707963 effort=7.5 velocity=3.1415927 -> lower=-1.5707963267948966 upper=1.5707963267948966 effort=7.5 velocity=3.1415927; origin xyz=0 0 0.0388 rpy=0 0 0 -> xyz=0.0334 0 0 rpy=0 0 0
- joint rj_dg_3_1: axis 1 0 0 -> 0 0 1; limit lower=-0.6108652 upper=0.6108652 effort=7.5 velocity=3.1415927 -> lower=-0.7330382858376184 upper=0.5759586531581288 effort=7.5 velocity=3.1415927; origin xyz=-0.0071 -0.0025 0.0701 rpy=0 0 0 -> xyz=0.0017 -0.005 0.08865 rpy=3.1416 -1.5708 0
- joint rj_dg_3_2: axis 0 1 0 -> 0 0 1; limit lower=0 upper=1.9547686 effort=7.5 velocity=3.1415927 -> lower=0 upper=2.2689280275926285 effort=7.5 velocity=3.1415927; origin xyz=0.01765 0 0.0265 rpy=0 0 0 -> xyz=0.02415 0 0.0126 rpy=1.5708 0 0
- joint rj_dg_3_3: axis 0 1 0 -> 0 0 1; limit lower=-1.5707963 upper=1.5707963 effort=7.5 velocity=3.1415927 -> lower=-1.5707963267948966 upper=1.5707963267948966 effort=7.5 velocity=3.1415927; origin xyz=0 0 0.0388 rpy=0 0 0 -> xyz=0.0334 0 0 rpy=0 0 0
- joint rj_dg_3_4: axis 0 1 0 -> 0 0 1; limit lower=-1.5707963 upper=1.5707963 effort=7.5 velocity=3.1415927 -> lower=-1.5707963267948966 upper=1.5707963267948966 effort=7.5 velocity=3.1415927; origin xyz=0 0 0.0388 rpy=0 0 0 -> xyz=0.0334 0 0 rpy=0 0 0
- joint rj_dg_4_1: axis 1 0 0 -> 0 0 1; limit lower=-0.418879 upper=0.6108652 effort=7.5 velocity=3.1415927 -> lower=-0.8377580409572782 upper=0.20943951023931956 effort=7.5 velocity=3.1415927; origin xyz=-0.0071 0.022 0.0621 rpy=0 0 0 -> xyz=0.0017 0.018 0.08065 rpy=3.1416 -1.5708 0
- joint rj_dg_4_2: axis 0 1 0 -> 0 0 1; limit lower=0 upper=1.9024088 effort=7.5 velocity=3.1415927 -> lower=0 upper=2.2165681500327987 effort=7.5 velocity=3.1415927; origin xyz=0.01765 0 0.0265 rpy=0 0 0 -> xyz=0.02415 0 0.0126 rpy=1.5708 0 0
- joint rj_dg_4_3: axis 0 1 0 -> 0 0 1; limit lower=-1.5707963 upper=1.5707963 effort=7.5 velocity=3.1415927 -> lower=-1.5707963267948966 upper=1.5707963267948966 effort=7.5 velocity=3.1415927; origin xyz=0 0 0.0388 rpy=0 0 0 -> xyz=0.0334 0 0 rpy=0 0 0
- joint rj_dg_4_4: axis 0 1 0 -> 0 0 1; limit lower=-1.5707963 upper=1.5707963 effort=7.5 velocity=3.1415927 -> lower=-1.5707963267948966 upper=1.5707963267948966 effort=7.5 velocity=3.1415927; origin xyz=0 0 0.0388 rpy=0 0 0 -> xyz=0.0334 0 0 rpy=0 0 0
- joint rj_dg_5_1: limit lower=-1.0471976 upper=0.0174533 effort=7.5 velocity=3.1415927 -> lower=-1.0471975511965976 upper=0 effort=7.5 velocity=3.1415927; origin xyz=0.0103 0.0195 0.0182 rpy=0 0 0 -> xyz=0.013 0.01805 0.0364 rpy=0 0 1.5708
- joint rj_dg_5_2: axis 1 0 0 -> 0 0 1; limit lower=-0.6108652 upper=0.418879 effort=7.5 velocity=3.1415927 -> lower=-1.5707963267948966 upper=0.6457718232379019 effort=7.5 velocity=3.1415927; origin xyz=0 0.028 0.0381 rpy=0 0 0 -> xyz=0.02445 0 0.0307 rpy=1.5708 0 0
- joint rj_dg_5_3: axis 0 1 0 -> 0 0 1; limit lower=-1.5707963 upper=1.5707963 effort=7.5 velocity=3.1415927 -> lower=-1.5707963267948966 upper=1.5707963267948966 effort=7.5 velocity=3.1415927; origin xyz=0 0 0.031 rpy=0 0 0 -> xyz=0 0.0272 0 rpy=1.5708 0 1.5708
- joint rj_dg_5_4: axis 0 1 0 -> 0 0 1; limit lower=-1.5707963 upper=1.5707963 effort=7.5 velocity=3.1415927 -> lower=-1.5707963267948966 upper=1.5707963267948966 effort=7.5 velocity=3.1415927; origin xyz=0 0 0.0388 rpy=0 0 0 -> xyz=0.0334 0 0 rpy=0 0 0
- joint rl_dg_1_tip_joint: origin xyz=0 -0.0363 0 rpy=0 0 0 -> xyz=0.0289 0 0 rpy=0 0 0
- joint rl_dg_2_tip_joint: origin xyz=0 0 0.0255 rpy=0 0 0 -> xyz=0.018 0 0 rpy=0 0 0
- joint rl_dg_3_tip_joint: origin xyz=0 0 0.0255 rpy=0 0 0 -> xyz=0.018 0 0 rpy=0 0 0
- joint rl_dg_4_tip_joint: origin xyz=0 0 0.0255 rpy=0 0 0 -> xyz=0.018 0 0 rpy=0 0 0
- joint rl_dg_5_tip_joint: origin xyz=0 0 0.0363 rpy=0 0 0 -> xyz=0.0289 0 0 rpy=0 0 0

File: source/FABRICS/src/fabrics_sim/models/robots/urdf/openarm_tesollo_sensor/openarm_tesollo_sensor.urdf (robot description, URDF)
Before this commit: robot openarm_tesollo_sensor, 63 links, 62 joints
Joints:
- joint palm_link_joint: origin xyz=0 3e-07 0.0685 rpy=0. 0. -1.5707964 -> xyz=0. 0.0000003 0.1333695 rpy=0. 0. -1.5707964
- joint rj_dg_1_1: axis 0 0 1 -> 1. 0. 0.; limit lower=-1.5707963267948966 upper=1.5707963267948966 effort=7.5 velocity=3.1415927 -> lower=-0.3839724 upper=0.8901179 effort=7.5 velocity=3.1415927; origin xyz=0.0017 0.018 0.0298 rpy=1.5708 0 1.5708 -> xyz=-0.0162 0.019 0.0128 rpy=0. 0. 0.
- joint rj_dg_1_2: axis 0 0 1 -> 0. 0. 1.; limit lower=-2.670353755551324 upper=0 effort=7.5 velocity=3.1415927 -> lower=-3.1415927 upper=0. effort=7.5 velocity=3.1415927; origin xyz=0 0 0.0262 rpy=-1.5708 0 0 -> xyz=0.04195 0. 0.  rpy=0. 0. 0.
- joint rj_dg_1_3: axis 0 0 1 -> 1. 0. 0.; limit lower=-1.5707963267948966 upper=1.5707963267948966 effort=7.5 velocity=3.1415927 -> lower=-1.5707963 upper=1.5707963 effort=7.5 velocity=3.1415927; origin xyz=0.0381 0 0 rpy=1.5708 0 0 -> xyz=0. 0.031 0.  rpy=0. 0. 0.
- joint rj_dg_1_4: axis 0 0 1 -> 1. 0. 0.; limit lower=-1.5707963267948966 upper=1.5707963267948966 effort=7.5 velocity=3.1415927 -> lower=-1.5707963 upper=1.5707963 effort=7.5 velocity=3.1415927; origin xyz=0.0334 0 0 rpy=0 0 0 -> xyz=0. 0.0388 0.  rpy=0. 0. 0.
- joint rj_dg_1_tip: origin xyz=0.0289 0 0 rpy=0 0 0 -> xyz=0. 0.0363 0. rpy=0. 0. 0.
- joint rj_dg_2_1: axis 0 0 1 -> 1. 0. 0.; limit lower=-0.8377580409572782 upper=0.2617993877991494 effort=7.5 velocity=3.1415927 -> lower=-0.418879 upper=0.6108652 effort=7.5 velocity=3.1415927; origin xyz=0.0017 0.028 0.08365 rpy=3.1416 -1.5708 0 -> xyz=-0.0071 0.027 0.0661 rpy=0. 0. 0.
- joint rj_dg_2_2: axis 0 0 -1 -> 0. 1. 0.; limit lower=0 upper=2.199114857512855 effort=7.5 velocity=3.1415927 -> lower=0. upper=2.0071286 effort=7.5 velocity=3.1415927; origin xyz=0.02415 0 0.0126 rpy=-1.5708 0 0 -> xyz=0.01765 0. 0.0265  rpy=0. 0. 0.
- joint rj_dg_2_3: axis 0 0 1 -> 0. 1. 0.; limit lower=-1.5707963267948966 upper=1.5707963267948966 effort=7.5 velocity=3.1415927 -> lower=-1.5707963 upper=1.5707963 effort=7.5 velocity=3.1415927; origin xyz=0.0334 0 0 rpy=3.1416 0 0 -> xyz=0. 0. 0.0388 rpy=0. 0. 0.
- joint rj_dg_2_4: axis 0 0 1 -> 0. 1. 0.; limit lower=-1.5707963267948966 upper=1.5707963267948966 effort=7.5 velocity=3.1415927 -> lower=-1.5707963 upper=1.5707963 effort=7.5 velocity=3.1415927; origin xyz=0.0334 0 0 rpy=0 0 0 -> xyz=0. 0. 0.0388 rpy=0. 0. 0.
- joint rj_dg_2_tip: origin xyz=0.018 0 0 rpy=0 0 0 -> xyz=0. 0. 0.0255 rpy=0. 0. 0.
- joint rj_dg_3_1: axis 0 0 1 -> 1. 0. 0.; limit lower=-0.5759586531581288 upper=0.7330382858376184 effort=7.5 velocity=3.1415927 -> lower=-0.6108652 upper=0.6108652 effort=7.5 velocity=3.1415927; origin xyz=0.0017 0.005 0.08865 rpy=3.1416 -1.5708 0 -> xyz=-0.0071 0.0025 0.0701 rpy=0. 0. 0.
- joint rj_dg_3_2: axis 0 0 -1 -> 0. 1. 0.; limit lower=0 upper=2.2689280275926285 effort=7.5 velocity=3.1415927 -> lower=0. upper=1.9547686 effort=7.5 velocity=3.1415927; origin xyz=0.02415 0 0.0126 rpy=-1.5708 0 0 -> xyz=0.01765 0. 0.0265  rpy=0. 0. 0.
- joint rj_dg_3_3: axis 0 0 1 -> 0. 1. 0.; limit lower=-1.5707963267948966 upper=1.5707963267948966 effort=7.5 velocity=3.1415927 -> lower=-1.5707963 upper=1.5707963 effort=7.5 velocity=3.1415927; origin xyz=0.0334 0 0 rpy=3.1416 0 0 -> xyz=0. 0. 0.0388 rpy=0. 0. 0.
- joint rj_dg_3_4: axis 0 0 1 -> 0. 1. 0.; limit lower=-1.5707963267948966 upper=1.5707963267948966 effort=7.5 velocity=3.1415927 -> lower=-1.5707963 upper=1.5707963 effort=7.5 velocity=3.1415927; origin xyz=0.0334 0 0 rpy=0 0 0 -> xyz=0. 0. 0.0388 rpy=0. 0. 0.
- joint rj_dg_3_tip: origin xyz=0.018 0 0 rpy=0 0 0 -> xyz=0. 0. 0.0255 rpy=0. 0. 0.
- joint rj_dg_4_1: axis 0 0 1 -> 1. 0. 0.; limit lower=-0.20943951023931956 upper=0.8377580409572782 effort=7.5 velocity=3.1415927 -> lower=-0.6108652 upper=0.418879 effort=7.5 velocity=3.1415927; origin xyz=0.0013 -0.018 0.08065 rpy=3.1416 -1.5708 0 -> xyz=-0.0071 -0.022 0.0621 rpy=0. 0. 0.
- joint rj_dg_4_2: axis 0 0 -1 -> 0. 1. 0.; limit lower=0 upper=2.2165681500327987 effort=7.5 velocity=3.1415927 -> lower=0. upper=1.9024088 effort=7.5 velocity=3.1415927; origin xyz=0.02415 0 0.0126 rpy=-1.5708 0 0 -> xyz=0.01765 0. 0.0265  rpy=0. 0. 0.
- joint rj_dg_4_3: axis 0 0 1 -> 0. 1. 0.; limit lower=-1.5707963267948966 upper=1.5707963267948966 effort=7.5 velocity=3.1415927 -> lower=-1.5707963 upper=1.5707963 effort=7.5 velocity=3.1415927; origin xyz=0.0334 0 0 rpy=3.1416 0 0 -> xyz=0. 0. 0.0388 rpy=0. 0. 0.
- joint rj_dg_4_4: axis 0 0 1 -> 0. 1. 0.; limit lower=-1.5707963267948966 upper=1.5707963267948966 effort=7.5 velocity=3.1415927 -> lower=-1.5707963 upper=1.5707963 effort=7.5 velocity=3.1415927; origin xyz=0.0334 0 0 rpy=0 0 0 -> xyz=0. 0. 0.0388 rpy=0. 0. 0.
- joint rj_dg_4_tip: origin xyz=0.018 0 0 rpy=0 0 0 -> xyz=0. 0. 0.0255 rpy=0. 0. 0.
- joint rj_dg_5_1: axis 0 0 1 -> 0. 0. 1.; limit lower=0 upper=1.0471975511965976 effort=7.5 velocity=3.1415927 -> lower=-0.0174533 upper=1.0471976 effort=7.5 velocity=3.1415927; origin xyz=0.013 -0.01805 0.0364 rpy=0 0 -1.5708 -> xyz=0.0103 -0.0195 0.0182 rpy=0. 0. 0.
- joint rj_dg_5_2: axis 0 0 1 -> 1. 0. 0.; limit lower=-0.6457718232379019 upper=1.5707963267948966 effort=7.5 velocity=3.1415927 -> lower=-0.418879 upper=0.6108652 effort=7.5 velocity=3.1415927; origin xyz=0.02445 0 0.0307 rpy=-1.5708 0 0 -> xyz=0. -0.028 0.0381 rpy=0. 0. 0.
- joint rj_dg_5_3: axis 0 0 1 -> 0. 1. 0.; limit lower=-1.5707963267948966 upper=1.5707963267948966 effort=7.5 velocity=3.1415927 -> lower=-1.5707963 upper=1.5707963 effort=7.5 velocity=3.1415927; origin xyz=0 -0.0272 0 rpy=1.5708 0 -1.5708 -> xyz=0. 0. 0.031 rpy=0. 0. 0.
- joint rj_dg_5_4: axis 0 0 1 -> 0. 1. 0.; limit lower=-1.5707963267948966 upper=1.5707963267948966 effort=7.5 velocity=3.1415927 -> lower=-1.5707963 upper=1.5707963 effort=7.5 velocity=3.1415927; origin xyz=0.0334 0 0 rpy=0 0 0 -> xyz=0. 0. 0.0388 rpy=0. 0. 0.
- joint rj_dg_5_tip: origin xyz=0.0289 0 0 rpy=0 0 0 -> xyz=0. 0. 0.0363 rpy=0. 0. 0.
