Commit message: feat(fabric): graft real r_hl_palm_sensor + IK axis points into rh56f1 urdf (right)
Tesollo palm_* 가상프레임(위치 3.4cm·자세 90° 어긋남) 제거, 참고 URDF 실기하로
palm_sensor 체인 + 축점 6개 graft. FK 정합 게이트 right PASS(0mm/0deg).

Co-Authored-By: Claude Opus 4.8 <noreply@anthropic.com>
Claude-Session: https://claude.ai/code/session_01BBFhucoTqrJR2pWGN5z87h

File: source/FABRICS/src/fabrics_sim/models/robots/urdf/openarm_rh56f1/openarm_rh56f1.urdf (robot description, URDF)
Before this commit: robot openarm_rh56f1, 49 links, 48 joints
Links:
- removed link palm_center
- removed link palm_link
- removed link palm_link_sphere2
- removed link palm_x
- removed link palm_x_neg
- removed link palm_y
- removed link palm_y_neg
- removed link palm_z
- removed link palm_z_neg
- added link ps_r_x, mass 0.001
- added link ps_r_x_neg, mass 0.001
- added link ps_r_y, mass 0.001
- added link ps_r_y_neg, mass 0.001
- added link ps_r_z, mass 0.001
- added link ps_r_z_neg, mass 0.001
- added link r_hl_palm_sensor, mass 0.001
- added link rh56f1_right_palm_1, mass 0.001
- added link rh56f1_right_palm_2, mass 0.001
Joints:
- removed joint palm_center_joint
- removed joint palm_link_joint
- removed joint palm_link_joint_sphere2
- removed joint palm_x_joint
- removed joint palm_x_neg_joint
- removed joint palm_y_joint
- removed joint palm_y_neg_joint
- removed joint palm_z_joint
- removed joint palm_z_neg_joint
- added joint ps_r_x_joint: type fixed, parent r_hl_palm_sensor, child ps_r_x, origin xyz=0.25 0 0 rpy=0 0 0
- added joint ps_r_x_neg_joint: type fixed, parent r_hl_palm_sensor, child ps_r_x_neg, origin xyz=-0.25 0 0 rpy=0 0 0
- added joint ps_r_y_joint: type fixed, parent r_hl_palm_sensor, child ps_r_y, origin xyz=0 0.25 0 rpy=0 0 0
- added joint ps_r_y_neg_joint: type fixed, parent r_hl_palm_sensor, child ps_r_y_neg, origin xyz=0 -0.25 0 rpy=0 0 0
- added joint ps_r_z_joint: type fixed, parent r_hl_palm_sensor, child ps_r_z, origin xyz=0 0 0.25 rpy=0 0 0
- added joint ps_r_z_neg_joint: type fixed, parent r_hl_palm_sensor, child ps_r_z_neg, origin xyz=0 0 -0.25 rpy=0 0 0
- added joint r_hl_palm_sensor_fixed_joint: type fixed, parent rh56f1_right_palm_2, child r_hl_palm_sensor, origin xyz=0.0159401947506102 -0.00135045394126701 0.0737460952299602 rpy=1.5707963267949 0 1.5707963267949
- added joint rh56f1_right_palm_1_fixed_joint: type fixed, parent rh56f1_right_base_link, child rh56f1_right_palm_1, origin xyz=0 0 0.0305 rpy=0 0 0
- added joint rh56f1_right_palm_2_fixed_joint: type fixed, parent rh56f1_right_palm_1, child rh56f1_right_palm_2, origin xyz=0 0 0 rpy=0 0 0

Commit message: feat(fabric): regenerate rh56f1 urdf from _rl source, bimanual 26 DOF
방향전환: Tesollo 팔 복사 폐기 → Isaac USD 와 동일한 _rl URDF 단일 소스.
- cspace 26: [r_arm7, r_hand6, l_arm7, l_hand6], drive 순서 정합
- 양쪽 r_hl/l_hl_palm_sensor + IK 축점(ps_r/l_*)
- FK 정합 both PASS 0mm/0deg (오른팔 base 6.4cm 오차 해소)

Co-Authored-By: Claude Opus 4.8 <noreply@anthropic.com>
Claude-Session: https://claude.ai/code/session_01BBFhucoTqrJR2pWGN5z87h

File: source/FABRICS/src/fabrics_sim/models/robots/urdf/openarm_rh56f1/openarm_rh56f1.urdf (robot description, URDF)
Before this commit: robot openarm_rh56f1, 49 links, 48 joints
Links:
- removed link openarm
- removed link openarm_right_link1
- removed link openarm_right_link2
- removed link openarm_right_link2_sphere2
- removed link openarm_right_link2_sphere3
- removed link openarm_right_link3
- removed link openarm_right_link4
- removed link openarm_right_link4_sphere2
- removed link openarm_right_link4_sphere3
- removed link openarm_right_link5
- removed link openarm_right_link6
- removed link openarm_right_link6_sphere2
- removed link openarm_right_link7
- removed link rh56f1_right_base_link
- removed link rh56f1_right_palm_1
- removed link rh56f1_right_palm_2
- removed link rh56f1_right_right_index_1
- removed link rh56f1_right_right_index_2
- removed link rh56f1_right_right_little_1
- removed link rh56f1_right_right_little_2
- removed link rh56f1_right_right_middle_1
- removed link rh56f1_right_right_middle_2
- removed link rh56f1_right_right_ring_1
- removed link rh56f1_right_right_ring_2
- removed link rh56f1_right_right_thumb_1
- removed link rh56f1_right_right_thumb_2
- removed link rh56f1_right_right_thumb_3
- removed link rh56f1_right_right_thumb_4
- removed link rh56f1_sphere_index
- removed link rh56f1_sphere_little
- removed link rh56f1_sphere_middle
- removed link rh56f1_sphere_ring
- removed link rh56f1_sphere_thumb
- removed link rh56f1_tip_index
- removed link rh56f1_tip_little
- removed link rh56f1_tip_middle
- removed link rh56f1_tip_ring
- removed link rh56f1_tip_thumb
- removed link world
- removed link world_body_sphere1
- removed link world_body_sphere2
- removed link world_body_sphere3
- added link body_link, mass 0.001
- added link l_al_0, mass 0.001
- added link l_al_1, mass 0.001
- added link l_al_2, mass 0.001
- added link l_al_3, mass 0.001
- added link l_al_4, mass 0.001
- added link l_al_5, mass 0.001
- added link l_al_6, mass 0.001
- added link l_al_7, mass 0.001
- added link l_hl_base, mass 0.001
- added link l_hl_index_1, mass 0.001
- added link l_hl_index_2, mass 0.001
- added link l_hl_index_tip, mass 0.001
- added link l_hl_middle_1, mass 0.001
- added link l_hl_middle_2, mass 0.001
- added link l_hl_middle_tip, mass 0.001
- added link l_hl_palm_1, mass 0.001
- added link l_hl_palm_2, mass 0.001
- added link l_hl_palm_3, mass 0.001
- added link l_hl_palm_sensor, mass 0.001
- added link l_hl_pinky_1, mass 0.001
- added link l_hl_pinky_2, mass 0.001
- added link l_hl_pinky_tip, mass 0.001
- added link l_hl_ring_1, mass 0.001
- added link l_hl_ring_2, mass 0.001
- added link l_hl_ring_tip, mass 0.001
- added link l_hl_thumb_1, mass 0.001
- added link l_hl_thumb_2, mass 0.001
- added link l_hl_thumb_3, mass 0.001
- added link l_hl_thumb_4, mass 0.001
- added link l_hl_thumb_tip, mass 0.001
- added link l_sphere_index, mass 0.001
- added link l_sphere_middle, mass 0.001
- added link l_sphere_pinky, mass 0.001
- added link l_sphere_ring, mass 0.001
- added link l_sphere_thumb, mass 0.001
- added link ps_l_x, mass 0.001
- added link ps_l_x_neg, mass 0.001
- added link ps_l_y, mass 0.001
- added link ps_l_y_neg, mass 0.001
- added link ps_l_z, mass 0.001
- added link ps_l_z_neg, mass 0.001
- added link r_al_0, mass 0.001
- added link r_al_1, mass 0.001
- added link r_al_2, mass 0.001
- added link r_al_3, mass 0.001
- added link r_al_4, mass 0.001
- added link r_al_5, mass 0.001
- added link r_al_6, mass 0.001
- added link r_al_7, mass 0.001
- added link r_hl_base, mass 0.001
- added link r_hl_index_1, mass 0.001
- added link r_hl_index_2, mass 0.001
- added link r_hl_index_tip, mass 0.001
- added link r_hl_middle_1, mass 0.001
- added link r_hl_middle_2, mass 0.001
- added link r_hl_middle_tip, mass 0.001
- added link r_hl_palm_1, mass 0.001
- added link r_hl_palm_2, mass 0.001
- added link r_hl_palm_3, mass 0.001
- added link r_hl_pinky_1, mass 0.001
- added link r_hl_pinky_2, mass 0.001
- added link r_hl_pinky_tip, mass 0.001
- added link r_hl_ring_1, mass 0.001
- added link r_hl_ring_2, mass 0.001
- added link r_hl_ring_tip, mass 0.001
- added link r_hl_thumb_1, mass 0.001
- added link r_hl_thumb_2, mass 0.001
- added link r_hl_thumb_3, mass 0.001
- added link r_hl_thumb_4, mass 0.001
- added link r_hl_thumb_tip, mass 0.001
- added link r_sphere_index, mass 0.001
- added link r_sphere_middle, mass 0.001
- added link r_sphere_pinky, mass 0.001
- added link r_sphere_ring, mass 0.001
- added link r_sphere_thumb, mass 0.001
Joints:
- removed joint openarm_right_joint1
- removed joint openarm_right_joint2
- removed joint openarm_right_joint3
- removed joint openarm_right_joint4
- removed joint openarm_right_joint5
- removed joint openarm_right_joint6
- removed joint openarm_right_joint7
- removed joint openarm_right_link2_joint_sphere2
- removed joint openarm_right_link2_joint_sphere3
- removed joint openarm_right_link4_joint_sphere2
- removed joint openarm_right_link4_joint_sphere3
- removed joint openarm_right_link6_joint_sphere2
- removed joint r_hl_palm_sensor_fixed_joint
- removed joint rh56f1_right_base_joint
- removed joint rh56f1_right_palm_1_fixed_joint
- removed joint rh56f1_right_palm_2_fixed_joint
- removed joint rh56f1_right_right_index_1_joint
- removed joint rh56f1_right_right_index_2_joint
- removed joint rh56f1_right_right_little_1_joint
- removed joint rh56f1_right_right_little_2_joint
- removed joint rh56f1_right_right_middle_1_joint
- removed joint rh56f1_right_right_middle_2_joint
- removed joint rh56f1_right_right_ring_1_joint
- removed joint rh56f1_right_right_ring_2_joint
- removed joint rh56f1_right_right_thumb_1_joint
- removed joint rh56f1_right_right_thumb_2_joint
- removed joint rh56f1_right_right_thumb_3_joint
- removed joint rh56f1_right_right_thumb_4_joint
- removed joint rh56f1_sphere_index_joint
- removed joint rh56f1_sphere_little_joint
- removed joint rh56f1_sphere_middle_joint
- removed joint rh56f1_sphere_ring_joint
- removed joint rh56f1_sphere_thumb_joint
- removed joint rh56f1_tip_index_joint
- removed joint rh56f1_tip_little_joint
- removed joint rh56f1_tip_middle_joint
- removed joint rh56f1_tip_ring_joint
- removed joint rh56f1_tip_thumb_joint
- removed joint root_joint
- removed joint world_body_joint_sphere1
- removed joint world_body_joint_sphere2
- removed joint world_body_joint_sphere3
- added joint l_aj_1: type revolute, parent l_al_0, child l_al_1, origin xyz=0.0 0.0 0.0625 rpy=0 0 0, axis 0 0 1, limit lower=-3.490659 upper=1.3962629999999998 effort=5 velocity=2
- added joint l_aj_2: type revolute, parent l_al_1, child l_al_2, origin xyz=-0.0301 0.0 0.06 rpy=-1.57079632679 0 0, axis -1 0 0, limit lower=-3.3161253267948965 upper=0.17453267320510335 effort=5 velocity=2
- added joint l_aj_3: type revolute, parent l_al_2, child l_al_3, origin xyz=0.0301 0.0 0.06625 rpy=0 0 0, axis 0 0 1, limit lower=-1.570796 upper=1.570796 effort=5 velocity=2
- added joint l_aj_4: type revolute, parent l_al_3, child l_al_4, origin xyz=-0.0 0.0315 0.15375 rpy=0 0 0, axis 0 1 0, limit lower=0.0 upper=2.443461 effort=5 velocity=2
- added joint l_aj_5: type revolute, parent l_al_4, child l_al_5, origin xyz=0.0 -0.0315 0.0955 rpy=0 0 0, axis 0 0 1, limit lower=-1.570796 upper=1.570796 effort=5 velocity=2
- added joint l_aj_6: type revolute, parent l_al_5, child l_al_6, origin xyz=0.0375 0.0 0.1205 rpy=0 0 0, axis 1 0 0, limit lower=-0.785398 upper=0.785398 effort=5 velocity=2
- added joint l_aj_7: type revolute, parent l_al_6, child l_al_7, origin xyz=-0.0375 0.0 0.0 rpy=0 0 0, axis 0 -1 0, limit lower=-1.570796 upper=1.570796 effort=5 velocity=2
- added joint l_aj_base: type fixed, parent body_link, child l_al_0, origin xyz=0.0 0.031 0.698 rpy=-1.5708 0 0
- added joint l_hj_index_1: type revolute, parent l_hl_base, child l_hl_index_1, origin xyz=0.00070753 -0.034377 0.13554 rpy=1.6319 0 0, axis 0 0 -1, limit lower=0 upper=1.5285593588966337 effort=5 velocity=2
- added joint l_hj_index_2: type fixed, parent l_hl_index_1, child l_hl_index_2, origin xyz=0.0031056 0.032854 -0.001 rpy=0 0 0
- added joint l_hj_index_tip: type fixed, parent l_hl_index_2, child l_hl_index_tip, origin xyz=0.0049188 0.039631 -0.006 rpy=-2.1925 1.5073 -1.8461
- added joint l_hj_middle_1: type revolute, parent l_hl_base, child l_hl_middle_1, origin xyz=0.00070746 -0.015767 0.13648 rpy=1.5708 0 0, axis 0 0 -1, limit lower=0 upper=1.5285593588966337 effort=5 velocity=2
- added joint l_hj_middle_2: type fixed, parent l_hl_middle_1, child l_hl_middle_2, origin xyz=0.0031056 0.032854 -0.001 rpy=0 0 0
- added joint l_hj_middle_tip: type fixed, parent l_hl_middle_2, child l_hl_middle_tip, origin xyz=0.0059647 0.042512 -0.0060998 rpy=-0.3273 1.5691 0
- added joint l_hj_mount: type fixed, parent l_al_7, child l_hl_base, origin xyz=0 0 0.0595695 rpy=0 0 1.5707964
- added joint l_hj_palm_1: type fixed, parent l_hl_base, child l_hl_palm_1, origin xyz=0 0 0.0305 rpy=0 0 0
- added joint l_hj_palm_2: type fixed, parent l_hl_palm_1, child l_hl_palm_2, origin xyz=0 0 0 rpy=0 0 0
- added joint l_hj_palm_3: type fixed, parent l_hl_palm_2, child l_hl_palm_3, origin xyz=0 0 0 rpy=0 0 0
- added joint l_hj_palm_sensor: type fixed, parent l_hl_palm_2, child l_hl_palm_sensor, origin xyz=0.01594 -0.0013505 0.073746 rpy=1.5708 0 1.5708
- added joint l_hj_pinky_1: type revolute, parent l_hl_base, child l_hl_pinky_1, origin xyz=0.00070753 0.021094 0.13531 rpy=1.4661 0 0, axis 0 0 -1, limit lower=0 upper=1.5285593588966337 effort=5 velocity=2
- added joint l_hj_pinky_2: type fixed, parent l_hl_pinky_1, child l_hl_pinky_2, origin xyz=0.0031057 0.032854 -0.001 rpy=0 0 0
- added joint l_hj_pinky_tip: type fixed, parent l_hl_pinky_2, child l_hl_pinky_tip, origin xyz=0.0051203 0.032544 -0.0063511 rpy=1.554 1.4608 1.8824
- added joint l_hj_ring_1: type revolute, parent l_hl_base, child l_hl_ring_1, origin xyz=0.00070746 0.0030876 0.13643 rpy=1.5184 0 0, axis 0 0 -1, limit lower=0 upper=1.5285593588966337 effort=5 velocity=2
- added joint l_hj_ring_2: type fixed, parent l_hl_ring_1, child l_hl_ring_2, origin xyz=0.0031056 0.032854 -0.001 rpy=0 0 0
- added joint l_hj_ring_tip: type fixed, parent l_hl_ring_2, child l_hl_ring_tip, origin xyz=0.0049188 0.039631 -0.006 rpy=1.5417 1.5157 1.889
- added joint l_hj_thumb_1: type revolute, parent l_hl_base, child l_hl_thumb_1, origin xyz=0.01836 -0.027241 0.070511 rpy=0 0 0, axis 8.7274E-05 0 1, limit lower=0 upper=2.0943951023931953 effort=5 velocity=2
- added joint l_hj_thumb_2: type revolute, parent l_hl_thumb_1, child l_hl_thumb_2, origin xyz=0.005034 -0.01349 -0.0049121 rpy=1.5707 0 -1.5708, axis 0 0 1, limit lower=0 upper=0.4745550236172582 effort=5 velocity=2
- added joint l_hj_thumb_3: type fixed, parent l_hl_thumb_2, child l_hl_thumb_3, origin xyz=0.033907 0.034601 -0.0029656 rpy=0 0 0
- added joint l_hj_thumb_4: type fixed, parent l_hl_thumb_3, child l_hl_thumb_4, origin xyz=0.01441 0.014648 0.0013 rpy=0 0 0
- added joint l_hj_thumb_tip: type fixed, parent l_hl_thumb_4, child l_hl_thumb_tip, origin xyz=0.016676 0.025314 0.0067577 rpy=1.8172 -1.5641 -3.1286
- added joint l_sphere_index_joint: type fixed, parent l_hl_index_1, child l_sphere_index, origin xyz=0 0.015 0 rpy=0 0 0
- added joint l_sphere_middle_joint: type fixed, parent l_hl_middle_1, child l_sphere_middle, origin xyz=0 0.015 0 rpy=0 0 0
- added joint l_sphere_pinky_joint: type fixed, parent l_hl_pinky_1, child l_sphere_pinky, origin xyz=0 0.015 0 rpy=0 0 0
- added joint l_sphere_ring_joint: type fixed, parent l_hl_ring_1, child l_sphere_ring, origin xyz=0 0.015 0 rpy=0 0 0
- added joint l_sphere_thumb_joint: type fixed, parent l_hl_thumb_2, child l_sphere_thumb, origin xyz=0 0.015 0 rpy=0 0 0
- added joint ps_l_x_joint: type fixed, parent l_hl_palm_sensor, child ps_l_x, origin xyz=0.25 0 0 rpy=0 0 0
- added joint ps_l_x_neg_joint: type fixed, parent l_hl_palm_sensor, child ps_l_x_neg, origin xyz=-0.25 0 0 rpy=0 0 0
- added joint ps_l_y_joint: type fixed, parent l_hl_palm_sensor, child ps_l_y, origin xyz=0 0.25 0 rpy=0 0 0
- added joint ps_l_y_neg_joint: type fixed, parent l_hl_palm_sensor, child ps_l_y_neg, origin xyz=0 -0.25 0 rpy=0 0 0
- added joint ps_l_z_joint: type fixed, parent l_hl_palm_sensor, child ps_l_z, origin xyz=0 0 0.25 rpy=0 0 0
- added joint ps_l_z_neg_joint: type fixed, parent l_hl_palm_sensor, child ps_l_z_neg, origin xyz=0 0 -0.25 rpy=0 0 0
- added joint r_aj_1: type revolute, parent r_al_0, child r_al_1, origin xyz=0.0 0.0 0.0625 rpy=0 0 0, axis 0 0 1, limit lower=-1.396263 upper=3.490659 effort=5 velocity=2
- added joint r_aj_2: type revolute, parent r_al_1, child r_al_2, origin xyz=-0.0301 0.0 0.06 rpy=1.57079632679 0 0, axis -1 0 0, limit lower=-0.17453267320510335 upper=3.3161253267948965 effort=5 velocity=2
- added joint r_aj_3: type revolute, parent r_al_2, child r_al_3, origin xyz=0.0301 0.0 0.06625 rpy=0 0 0, axis 0 0 1, limit lower=-1.570796 upper=1.570796 effort=5 velocity=2
- added joint r_aj_4: type revolute, parent r_al_3, child r_al_4, origin xyz=-0.0 0.0315 0.15375 rpy=0 0 0, axis 0 1 0, limit lower=0.0 upper=2.443461 effort=5 velocity=2
- added joint r_aj_5: type revolute, parent r_al_4, child r_al_5, origin xyz=0.0 -0.0315 0.0955 rpy=0 0 0, axis 0 0 1, limit lower=-1.570796 upper=1.570796 effort=5 velocity=2
- added joint r_aj_6: type revolute, parent r_al_5, child r_al_6, origin xyz=0.0375 0.0 0.1205 rpy=0 0 0, axis 1 0 0, limit lower=-0.785398 upper=0.785398 effort=5 velocity=2
- added joint r_aj_7: type revolute, parent r_al_6, child r_al_7, origin xyz=-0.0375 0.0 0.0 rpy=0 0 0, axis 0 1 0, limit lower=-1.570796 upper=1.570796 effort=5 velocity=2
- added joint r_aj_base: type fixed, parent body_link, child r_al_0, origin xyz=0.0 -0.031 0.698 rpy=1.5708 0 0
- added joint r_hj_index_1: type revolute, parent r_hl_base, child r_hl_index_1, origin xyz=0.00070751 0.034376 0.13554 rpy=1.5097 0 0, axis 0 0 -1, limit lower=0 upper=1.5285593588966337 effort=5 velocity=2
- added joint r_hj_index_2: type fixed, parent r_hl_index_1, child r_hl_index_2, origin xyz=0.0031056 0.032854 0.001 rpy=0 0 0
- added joint r_hj_index_tip: type fixed, parent r_hl_index_2, child r_hl_index_tip, origin xyz=0.0049188 0.039631 0.006 rpy=1.5446 1.5064 1.892
- added joint r_hj_middle_1: type revolute, parent r_hl_base, child r_hl_middle_1, origin xyz=0.00070746 0.015767 0.13648 rpy=1.5708 0 0, axis 0 0 -1, limit lower=0 upper=1.5285593588966337 effort=5 velocity=2
- added joint r_hj_middle_2: type fixed, parent r_hl_middle_1, child r_hl_middle_2, origin xyz=0.0031056 0.032854 0.001 rpy=0 0 0
- added joint r_hj_middle_tip: type fixed, parent r_hl_middle_2, child r_hl_middle_tip, origin xyz=0.0059647 0.042512 0.0060998 rpy=-0.3273 1.5691 0
- added joint r_hj_mount: type fixed, parent r_al_7, child r_hl_base, origin xyz=0 0.0000003 0.0595695 rpy=0 0 -1.5707964
- added joint r_hj_palm_1: type fixed, parent r_hl_base, child r_hl_palm_1, origin xyz=0 0 0.0305 rpy=0 0 0
- added joint r_hj_palm_2: type fixed, parent r_hl_palm_1, child r_hl_palm_2, origin xyz=0 0 0 rpy=0 0 0
- added joint r_hj_palm_3: type fixed, parent r_hl_palm_2, child r_hl_palm_3, origin xyz=0 0 0 rpy=0 0 0
- added joint r_hj_palm_sensor: type fixed, parent r_hl_palm_2, child r_hl_palm_sensor, origin xyz=0.0159401947506102 -0.00135045394126701 0.0737460952299602 rpy=1.5707963267949 0 1.5707963267949
- added joint r_hj_pinky_1: type revolute, parent r_hl_base, child r_hl_pinky_1, origin xyz=0.00070753 -0.021451 0.13527 rpy=1.6755 0 0, axis 0 0 -1, limit lower=0 upper=1.5285593588966337 effort=5 velocity=2
- added joint r_hj_pinky_2: type fixed, parent r_hl_pinky_1, child r_hl_pinky_2, origin xyz=0.0031057 0.032854 0.001 rpy=0 0 0
- added joint r_hj_pinky_tip: type fixed, parent r_hl_pinky_2, child r_hl_pinky_tip, origin xyz=0.0051203 0.032544 0.0059927 rpy=-1.5577 1.4597 -1.2296
- added joint r_hj_ring_1: type revolute, parent r_hl_base, child r_hl_ring_1, origin xyz=0.00070746 -0.0030876 0.13643 rpy=1.6232 0 0, axis 0 0 -1, limit lower=0 upper=1.5285593588966337 effort=5 velocity=2
- added joint r_hj_ring_2: type fixed, parent r_hl_ring_1, child r_hl_ring_2, origin xyz=0.0031056 0.032854 0.001 rpy=0 0 0
- added joint r_hj_ring_tip: type fixed, parent r_hl_ring_2, child r_hl_ring_tip, origin xyz=0.0049188 0.039631 0.006 rpy=-1.5409 1.5145 -1.1936
- added joint r_hj_thumb_1: type revolute, parent r_hl_base, child r_hl_thumb_1, origin xyz=0.01836 0.027241 0.070511 rpy=0 0 0, axis 8.7274E-05 0 -1, limit lower=0 upper=2.0943951023931953 effort=5 velocity=2
- added joint r_hj_thumb_2: type revolute, parent r_hl_thumb_1, child r_hl_thumb_2, origin xyz=0.0047995 0.013396 -0.0052536 rpy=1.5707 0 -1.5708, axis 0 0 -1, limit lower=0 upper=0.4745550236172582 effort=5 velocity=2
- added joint r_hj_thumb_3: type fixed, parent r_hl_thumb_2, child r_hl_thumb_3, origin xyz=-0.029155 0.03869 -0.0032 rpy=0 0 0
- added joint r_hj_thumb_4: type fixed, parent r_hl_thumb_3, child r_hl_thumb_4, origin xyz=-0.01441 0.014648 0.0013 rpy=0 0 0
- added joint r_hj_thumb_tip: type fixed, parent r_hl_thumb_4, child r_hl_thumb_tip, origin xyz=-0.017405 0.025196 0.0068001 rpy=-1.2971 1.5647 0.01425
- added joint r_sphere_index_joint: type fixed, parent r_hl_index_1, child r_sphere_index, origin xyz=0 0.015 0 rpy=0 0 0
- added joint r_sphere_middle_joint: type fixed, parent r_hl_middle_1, child r_sphere_middle, origin xyz=0 0.015 0 rpy=0 0 0
- added joint r_sphere_pinky_joint: type fixed, parent r_hl_pinky_1, child r_sphere_pinky, origin xyz=0 0.015 0 rpy=0 0 0
- added joint r_sphere_ring_joint: type fixed, parent r_hl_ring_1, child r_sphere_ring, origin xyz=0 0.015 0 rpy=0 0 0
- added joint r_sphere_thumb_joint: type fixed, parent r_hl_thumb_2, child r_sphere_thumb, origin xyz=0 0.015 0 rpy=0 0 0
