Commit message: feat(fabrics): fabric URDF 4종 재생성 — canonical RL URDF 파생 + manifest 신설
rl_ws/urdf 파이프라인 gen_fabric_urdfs.py 산출물(수기 편집본 → 생성본 전환).

- 팔 베이스 z 0.698→0.690: USD 는 07.29 head 교체 때 팔이 8mm 하강했는데
  구 fabric URDF 만 옛 높이였다. smoke 의 상시 palm 추종오차 8.0mm 가 정확히
  이 불일치였고, 재생성 후 좌·우 모두 0.6mm 로 감소 (13배 정밀화).
- bi_s_left: M-conjugation 미러 근사 → RL URDF l-체인 직접 생성(joint4/5
  y-부호 반전이 정답 — 미러 근사가 틀려 있었다). 좌·우 smoke 수치 완전 대칭.
- palm_center·자세·충돌 sphere·tip 가상 프레임 63개 보존, cspace finger-major
  순서를 manifest 로 명문화.

검증: probe_grasp_lift_fabric_smoke 좌·우 PASS (self_collisions+gravity ON,
추종 0.6mm · 컵 교란 0 · 접촉 PASS · 26k fps)

File: source/FABRICS/src/fabrics_sim/models/robots/urdf/openarm_rh56f1/openarm_rh56f1.urdf (robot description, URDF)
Before this commit: robot openarm_rh56f1, 83 links, 82 joints
Joints:
- joint l_aj_base: origin xyz=0.0 0.031 0.698 rpy=-1.5708 0 0 -> xyz=0 0.031 0.69 rpy=-1.5708 0 0
- joint r_aj_base: origin xyz=0.0 -0.031 0.698 rpy=1.5708 0 0 -> xyz=0 -0.031 0.69 rpy=1.5708 0 0

File: source/FABRICS/src/fabrics_sim/models/robots/urdf/openarm_tesollo_bi_s/openarm_tesollo_bi_s.urdf (robot description, URDF)
Before this commit: robot open_tesollo, 62 links, 61 joints
Joints:
- joint openarm_right_joint1: axis 0. 0. 1. -> 0 0 1; limit lower=-1.3962629 upper=3.4906588 effort=40. velocity=16.7546644 -> lower=-1.396263 upper=3.490659 effort=40. velocity=16.7546644; origin xyz=0. -0.0935 0.6979998 rpy=1.5708 0. 0.  -> xyz=0 -0.0935 0.68999977 rpy=1.5708 0 0
- joint openarm_right_joint2: axis 1. 0. 0. -> -1 0 0; limit lower=-0.1745327 upper=3.3161253 effort=40. velocity=16.7546644 -> lower=-0.174532673 upper=3.31612533 effort=40. velocity=16.7546644; origin xyz=-0.0301 0. 0.06  rpy=-1.5707963 0. 3.1415927 -> xyz=-0.0301 0 0.06 rpy=1.57079633 0 0
- joint openarm_right_joint3: axis 0. 0. 1. -> 0 0 1; limit lower=-1.5707959 upper=1.5707959 effort=27. velocity=5.4454257 -> lower=-1.570796 upper=1.570796 effort=27. velocity=5.4454257; origin xyz=-0.0301 -0. 0.06625 rpy=0. 0. 3.1415927 -> xyz=0.0301 0 0.06625 rpy=0 0 0
- joint openarm_right_joint4: axis 0. 1. 0. -> 0 1 0; limit lower=0. upper=2.4434607 effort=27. velocity=5.4454257 -> lower=0 upper=2.443461 effort=27. velocity=5.4454257; origin xyz=0. 0.0315 0.15375 rpy=0. 0. 0. -> xyz=0 0.0315 0.15375 rpy=0 0 0
- joint openarm_right_joint5: axis 0. 0. 1. -> 0 0 1; limit lower=-1.5707959 upper=1.5707959 effort=7. velocity=20.9439446 -> lower=-1.570796 upper=1.570796 effort=7. velocity=20.9439446; origin xyz=0. -0.0315 0.0955 rpy=0. 0. 0. -> xyz=0 -0.0315 0.0955 rpy=0 0 0
- joint openarm_right_joint6: axis 1. 0. 0. -> 1 0 0; origin xyz=0.0375 0. 0.1205 rpy=0. 0. 0. -> xyz=0.0375 0 0.1205 rpy=0 0 0
- joint openarm_right_joint7: axis 0. 1. 0. -> 0 1 0; limit lower=-1.5707959 upper=1.5707959 effort=7. velocity=20.9439446 -> lower=-1.570796 upper=1.570796 effort=7. velocity=20.9439446; origin xyz=-0.0375 0. 0.  rpy=0. 0. 0. -> xyz=-0.0375 0 0 rpy=0 0 0
- joint rj_dg_1_1: limit lower=-1.5707963267948966 upper=1.5707963267948966 effort=7.5 velocity=3.1415927 -> lower=-1.57079633 upper=1.57079633 effort=7.5 velocity=3.1415927
- joint rj_dg_1_2: limit lower=-2.670353755551324 upper=0 effort=7.5 velocity=3.1415927 -> lower=-2.67035376 upper=0 effort=7.5 velocity=3.1415927
- joint rj_dg_1_3: limit lower=-1.5707963267948966 upper=1.5707963267948966 effort=7.5 velocity=3.1415927 -> lower=-1.57079633 upper=1.57079633 effort=7.5 velocity=3.1415927
- joint rj_dg_1_4: limit lower=-1.5707963267948966 upper=1.5707963267948966 effort=7.5 velocity=3.1415927 -> lower=-1.57079633 upper=1.57079633 effort=7.5 velocity=3.1415927
- joint rj_dg_2_1: limit lower=-0.8377580409572782 upper=0.2617993877991494 effort=7.5 velocity=3.1415927 -> lower=-0.837758041 upper=0.261799388 effort=7.5 velocity=3.1415927
- joint rj_dg_2_2: limit lower=0 upper=2.199114857512855 effort=7.5 velocity=3.1415927 -> lower=0 upper=2.19911486 effort=7.5 velocity=3.1415927
- joint rj_dg_2_3: limit lower=-1.5707963267948966 upper=1.5707963267948966 effort=7.5 velocity=3.1415927 -> lower=-1.57079633 upper=1.57079633 effort=7.5 velocity=3.1415927
- joint rj_dg_2_4: limit lower=-1.5707963267948966 upper=1.5707963267948966 effort=7.5 velocity=3.1415927 -> lower=-1.57079633 upper=1.57079633 effort=7.5 velocity=3.1415927
- joint rj_dg_3_1: limit lower=-0.5759586531581288 upper=0.7330382858376184 effort=7.5 velocity=3.1415927 -> lower=-0.575958653 upper=0.733038286 effort=7.5 velocity=3.1415927
- joint rj_dg_3_2: limit lower=0 upper=2.2689280275926285 effort=7.5 velocity=3.1415927 -> lower=0 upper=2.26892803 effort=7.5 velocity=3.1415927
- joint rj_dg_3_3: limit lower=-1.5707963267948966 upper=1.5707963267948966 effort=7.5 velocity=3.1415927 -> lower=-1.57079633 upper=1.57079633 effort=7.5 velocity=3.1415927
- joint rj_dg_3_4: limit lower=-1.5707963267948966 upper=1.5707963267948966 effort=7.5 velocity=3.1415927 -> lower=-1.57079633 upper=1.57079633 effort=7.5 velocity=3.1415927
- joint rj_dg_4_1: limit lower=-0.20943951023931956 upper=0.8377580409572782 effort=7.5 velocity=3.1415927 -> lower=-0.20943951 upper=0.837758041 effort=7.5 velocity=3.1415927
- joint rj_dg_4_2: limit lower=0 upper=2.2165681500327987 effort=7.5 velocity=3.1415927 -> lower=0 upper=2.21656815 effort=7.5 velocity=3.1415927
- joint rj_dg_4_3: limit lower=-1.5707963267948966 upper=1.5707963267948966 effort=7.5 velocity=3.1415927 -> lower=-1.57079633 upper=1.57079633 effort=7.5 velocity=3.1415927
- joint rj_dg_4_4: limit lower=-1.5707963267948966 upper=1.5707963267948966 effort=7.5 velocity=3.1415927 -> lower=-1.57079633 upper=1.57079633 effort=7.5 velocity=3.1415927
- joint rj_dg_5_1: limit lower=0 upper=1.0471975511965976 effort=7.5 velocity=3.1415927 -> lower=0 upper=1.04719755 effort=7.5 velocity=3.1415927
- joint rj_dg_5_2: limit lower=-0.6457718232379019 upper=1.5707963267948966 effort=7.5 velocity=3.1415927 -> lower=-0.645771823 upper=1.57079633 effort=7.5 velocity=3.1415927
- joint rj_dg_5_3: limit lower=-1.5707963267948966 upper=1.5707963267948966 effort=7.5 velocity=3.1415927 -> lower=-1.57079633 upper=1.57079633 effort=7.5 velocity=3.1415927
- joint rj_dg_5_4: limit lower=-1.5707963267948966 upper=1.5707963267948966 effort=7.5 velocity=3.1415927 -> lower=-1.57079633 upper=1.57079633 effort=7.5 velocity=3.1415927

File: source/FABRICS/src/fabrics_sim/models/robots/urdf/openarm_tesollo_bi_s_left/openarm_tesollo_bi_s_left.urdf (robot description, URDF)
Before this commit: robot openarm_tesollo_bi_s_left, 62 links, 61 joints
Joints:
- joint openarm_right_joint1: limit lower=-3.4906588 upper=1.3962629 effort=40. velocity=16.7546644 -> lower=-3.490659 upper=1.396263 effort=40. velocity=16.7546644; origin xyz=0 0.0935 0.6979998 rpy=-1.5708 0 0 -> xyz=0 0.0935 0.68999977 rpy=-1.5708 0 0
- joint openarm_right_joint2: axis 1 0 0 -> -1 0 0; limit lower=-3.3161253 upper=0.1745327 effort=40. velocity=16.7546644 -> lower=-3.31612533 upper=0.174532673 effort=40. velocity=16.7546644; origin xyz=-0.0301 0 0.06 rpy=1.5707963 0 3.14159261 -> xyz=-0.0301 0 0.06 rpy=-1.57079633 0 0
- joint openarm_right_joint3: limit lower=-1.5707959 upper=1.5707959 effort=27. velocity=5.4454257 -> lower=-1.570796 upper=1.570796 effort=27. velocity=5.4454257; origin xyz=-0.0301 0 0.06625 rpy=0 0 3.14159261 -> xyz=0.0301 0 0.06625 rpy=0 0 0
- joint openarm_right_joint4: limit lower=0 upper=2.4434607 effort=27. velocity=5.4454257 -> lower=0 upper=2.443461 effort=27. velocity=5.4454257; origin xyz=0 -0.0315 0.15375 rpy=0 0 0 -> xyz=0 0.0315 0.15375 rpy=0 0 0
- joint openarm_right_joint5: limit lower=-1.5707959 upper=1.5707959 effort=7. velocity=20.9439446 -> lower=-1.570796 upper=1.570796 effort=7. velocity=20.9439446; origin xyz=0 0.0315 0.0955 rpy=0 0 0 -> xyz=0 -0.0315 0.0955 rpy=0 0 0
- joint openarm_right_joint7: limit lower=-1.5707959 upper=1.5707959 effort=7. velocity=20.9439446 -> lower=-1.570796 upper=1.570796 effort=7. velocity=20.9439446
- joint rj_dg_1_1: limit lower=-1.5707963267948966 upper=1.5707963267948966 effort=7.5 velocity=3.1415927 -> lower=-1.57079633 upper=1.57079633 effort=7.5 velocity=3.1415927
- joint rj_dg_1_2: limit lower=0 upper=2.670353755551324 effort=7.5 velocity=3.1415927 -> lower=0 upper=2.67035376 effort=7.5 velocity=3.1415927
- joint rj_dg_1_3: limit lower=-1.5707963267948966 upper=1.5707963267948966 effort=7.5 velocity=3.1415927 -> lower=-1.57079633 upper=1.57079633 effort=7.5 velocity=3.1415927
- joint rj_dg_1_4: limit lower=-1.5707963267948966 upper=1.5707963267948966 effort=7.5 velocity=3.1415927 -> lower=-1.57079633 upper=1.57079633 effort=7.5 velocity=3.1415927
- joint rj_dg_2_1: limit lower=-0.2617993877991494 upper=0.8377580409572782 effort=7.5 velocity=3.1415927 -> lower=-0.261799388 upper=0.837758041 effort=7.5 velocity=3.1415927
- joint rj_dg_2_2: limit lower=0 upper=2.199114857512855 effort=7.5 velocity=3.1415927 -> lower=0 upper=2.19911486 effort=7.5 velocity=3.1415927
- joint rj_dg_2_3: limit lower=-1.5707963267948966 upper=1.5707963267948966 effort=7.5 velocity=3.1415927 -> lower=-1.57079633 upper=1.57079633 effort=7.5 velocity=3.1415927
- joint rj_dg_2_4: limit lower=-1.5707963267948966 upper=1.5707963267948966 effort=7.5 velocity=3.1415927 -> lower=-1.57079633 upper=1.57079633 effort=7.5 velocity=3.1415927
- joint rj_dg_3_1: limit lower=-0.7330382858376184 upper=0.5759586531581288 effort=7.5 velocity=3.1415927 -> lower=-0.733038286 upper=0.575958653 effort=7.5 velocity=3.1415927
- joint rj_dg_3_2: limit lower=0 upper=2.2689280275926285 effort=7.5 velocity=3.1415927 -> lower=0 upper=2.26892803 effort=7.5 velocity=3.1415927
- joint rj_dg_3_3: limit lower=-1.5707963267948966 upper=1.5707963267948966 effort=7.5 velocity=3.1415927 -> lower=-1.57079633 upper=1.57079633 effort=7.5 velocity=3.1415927
- joint rj_dg_3_4: limit lower=-1.5707963267948966 upper=1.5707963267948966 effort=7.5 velocity=3.1415927 -> lower=-1.57079633 upper=1.57079633 effort=7.5 velocity=3.1415927
- joint rj_dg_4_1: limit lower=-0.8377580409572782 upper=0.20943951023931956 effort=7.5 velocity=3.1415927 -> lower=-0.837758041 upper=0.20943951 effort=7.5 velocity=3.1415927
- joint rj_dg_4_2: limit lower=0 upper=2.2165681500327987 effort=7.5 velocity=3.1415927 -> lower=0 upper=2.21656815 effort=7.5 velocity=3.1415927
- joint rj_dg_4_3: limit lower=-1.5707963267948966 upper=1.5707963267948966 effort=7.5 velocity=3.1415927 -> lower=-1.57079633 upper=1.57079633 effort=7.5 velocity=3.1415927
- joint rj_dg_4_4: limit lower=-1.5707963267948966 upper=1.5707963267948966 effort=7.5 velocity=3.1415927 -> lower=-1.57079633 upper=1.57079633 effort=7.5 velocity=3.1415927
- joint rj_dg_5_1: limit lower=-1.0471975511965976 upper=0 effort=7.5 velocity=3.1415927 -> lower=-1.04719755 upper=0 effort=7.5 velocity=3.1415927
- joint rj_dg_5_2: limit lower=-1.5707963267948966 upper=0.6457718232379019 effort=7.5 velocity=3.1415927 -> lower=-1.57079633 upper=0.645771823 effort=7.5 velocity=3.1415927
- joint rj_dg_5_3: limit lower=-1.5707963267948966 upper=1.5707963267948966 effort=7.5 velocity=3.1415927 -> lower=-1.57079633 upper=1.57079633 effort=7.5 velocity=3.1415927
- joint rj_dg_5_4: limit lower=-1.5707963267948966 upper=1.5707963267948966 effort=7.5 velocity=3.1415927 -> lower=-1.57079633 upper=1.57079633 effort=7.5 velocity=3.1415927
