Commit message: fix(fabrics): 좌팔 URDF palm helper 프레임 미러 제외 — attractor 7점 규약 유지

File: source/FABRICS/src/fabrics_sim/models/robots/urdf/openarm_tesollo_left/openarm_tesollo_left.urdf (robot description, URDF)
Before this commit: robot openarm_tesollo_left, 62 links, 61 joints
Joints:
- joint palm_x_joint: origin xyz=0.25 0 0 rpy=0 0 0 -> xyz=0.25 0. 0. rpy=0. 0. 0.
- joint palm_x_neg_joint: origin xyz=-0.25 0 0 rpy=0 0 0 -> xyz=-0.25 0. 0. rpy=0. 0. 0.
- joint palm_y_joint: origin xyz=0 -0.25 0 rpy=0 0 0 -> xyz=0. 0.25 0. rpy=0. 0. 0.
- joint palm_y_neg_joint: origin xyz=0 0.25 0 rpy=0 0 0 -> xyz=0. -0.25 0. rpy=0. 0. 0.
- joint palm_z_joint: origin xyz=0 0 0.25 rpy=0 0 0 -> xyz=0. 0. 0.25 rpy=0. 0. 0.
- joint palm_z_neg_joint: origin xyz=0 0 -0.25 rpy=0 0 0 -> xyz=0. 0. -0.25 rpy=0. 0. 0.
