Commit message: assets(cocktail): shaker 바닥면 있는 버전으로 재제작 (meshes/urdf/usda)
바닥면 없던 기존 shaker → 바닥면 포함 재생성. thick3mm/solid_envelope collision stl 정리.
※ grasp_v1은 visdex_objects/USD/shaker_body/shaker_body.usd(fix_shaker_asset 생성본)를
  사용하므로 현재 학습엔 미반영. 원본 백업·동기화용.

File: assets/cocktail/urdf/shaker_assembled.urdf (robot description, URDF)
Before this commit: robot cocktail_shaker_assembled, 1 links, 0 joints
Links:
- link shaker: mass 0.4993 -> 0.5460

File: assets/cocktail/urdf/shaker_body.urdf (robot description, URDF)
Before this commit: robot cocktail_shaker_body, 1 links, 0 joints
Links:
- link shaker_body: mass 0.2633 -> 0.2876

File: assets/cocktail/urdf/shaker_cap.urdf (robot description, URDF)
Before this commit: robot cocktail_shaker_cap, 1 links, 0 joints
Links:
- link shaker_cap: mass 0.0583 -> 0.0808
