Commit message: feat: 신규 로봇 USD(head 카메라) 교체 + 전 정책 head actuator group 추가
- sensor_rl/bi_rl/rh56f1 USD를 head 카메라(pan/tilt) 부착본으로 교체
  (s2r base 정합: origin=mount plate top, body_link 기준 팔 -8mm)
- head_j_pan/tilt(revolute)가 DOF로 잡히므로 10개 정책 actuator에 head_camera group 추가
  (커버리지 없으면 크래시/자유회전; stiffness 400/80으로 기본각 0 hold)
- obs/action은 이름 기반(joint_names.index)이라 head 미포함 유지 → 차원 불변

Co-Authored-By: Claude Opus 4.8 <noreply@anthropic.com>
Claude-Session: https://claude.ai/code/session_01GqgiSFhpMVqs48Qb2jAb13

File: assets/robot/openarm_bi_rh56f1_rl/openarm_bi_rh56f1_rl.urdf (robot description, URDF)
Before this commit: robot openarm_bi_rh56f1_rl, 72 links, 71 joints
Links:
- added link head_base, mass 0.109629; collision mesh filename=file:///home/user/rl_ws/urdf/vendor/head_realsense_d435i/me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 scale=0.001 0.001 0.001; visual mesh filename=file:///home/user/rl_ws/urdf/vendor/head_realsense_d435i/me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 scale=0.001 0.001 0.001
- added link head_cam_view
- added link head_camera, mass 0.065101; collision mesh filename=file:///home/user/rl_ws/urdf/vendor/head_realsense_d435i/me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 scale=0.001 0.001 0.001; visual mesh filename=file:///home/user/rl_ws/urdf/vendor/head_realsense_d435i/me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 scale=0.001 0.001 0.001
- added link head_mid, mass 0.017073; collision mesh filename=file:///home/user/rl_ws/urdf/vendor/head_realsense_d435i/me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 scale=0.001 0.001 0.001; visual mesh filename=file:///home/user/rl_ws/urdf/vendor/head_realsense_d435i/me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 scale=0.001 0.001 0.001
- link body_link: geometry collision mesh filename=file:///home/user/rl_ws/urdf/generated/rl/meshes/body_link0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 scale=0.001 0.001 0.001; visual mesh filename=file:///home/user/rl_ws/urdf/generated/rl/meshes/body_link0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 scale=0.001 0.001 0.001
Joints:
- added joint head_j_cam_view: type fixed, parent head_camera, child head_cam_view, origin xyz=0.0147 0.0145 0.0365 rpy=0 0 0
- added joint head_j_mount: type fixed, parent body_link, child head_base, origin xyz=0 0 0.750 rpy=0 0 0
- added joint head_j_pan: type revolute, parent head_base, child head_mid, origin xyz=0.0225 0 0.0385 rpy=0 0 0, axis 0 0 -1, limit lower=-1.5708 upper=1.5708 effort=1.0 velocity=6.0
- added joint head_j_tilt: type revolute, parent head_mid, child head_camera, origin xyz=0 -0.0145 0.0275 rpy=0 0 0, axis 0 1 0, limit lower=-1.570796 upper=1.570796 effort=1.0 velocity=6.0
- joint l_aj_base: origin xyz=0.0 0.031 0.698 rpy=-1.5708 0 0 -> xyz=0 0.031 0.69 rpy=-1.5708 0 0
- joint r_aj_base: origin xyz=0.0 -0.031 0.698 rpy=1.5708 0 0 -> xyz=0 -0.031 0.69 rpy=1.5708 0 0

File: assets/robot/openarm_tesollo_bi_rl/openarm_tesollo_bi_rl.urdf (robot description, URDF)
Before this commit: robot openarm_dual_tesollo_rl, 80 links, 79 joints
Links:
- added link head_base, mass 0.109629; collision mesh filename=file:///home/user/rl_ws/urdf/vendor/head_realsense_d435i/me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 scale=0.001 0.001 0.001; visual mesh filename=file:///home/user/rl_ws/urdf/vendor/head_realsense_d435i/me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 scale=0.001 0.001 0.001
- added link head_cam_view
- added link head_camera, mass 0.065101; collision mesh filename=file:///home/user/rl_ws/urdf/vendor/head_realsense_d435i/me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 scale=0.001 0.001 0.001; visual mesh filename=file:///home/user/rl_ws/urdf/vendor/head_realsense_d435i/me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 scale=0.001 0.001 0.001
- added link head_mid, mass 0.017073; collision mesh filename=file:///home/user/rl_ws/urdf/vendor/head_realsense_d435i/me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 scale=0.001 0.001 0.001; visual mesh filename=file:///home/user/rl_ws/urdf/vendor/head_realsense_d435i/me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 scale=0.001 0.001 0.001
- link body_link: geometry collision mesh filename=file:///home/user/rl_ws/urdf/generated/rl/meshes/body_link0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 scale=0.001 0.001 0.001; visual mesh filename=file:///home/user/rl_ws/urdf/generated/rl/meshes/body_link0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 scale=0.001 0.001 0.001
Joints:
- added joint head_j_cam_view: type fixed, parent head_camera, child head_cam_view, origin xyz=0.0147 0.0145 0.0365 rpy=0 0 0
- added joint head_j_mount: type fixed, parent body_link, child head_base, origin xyz=0 0 0.750 rpy=0 0 0
- added joint head_j_pan: type revolute, parent head_base, child head_mid, origin xyz=0.0225 0 0.0385 rpy=0 0 0, axis 0 0 -1, limit lower=-1.5708 upper=1.5708 effort=1.0 velocity=6.0
- added joint head_j_tilt: type revolute, parent head_mid, child head_camera, origin xyz=0 -0.0145 0.0275 rpy=0 0 0, axis 0 1 0, limit lower=-1.570796 upper=1.570796 effort=1.0 velocity=6.0
- joint l_aj_base: origin xyz=0.0 0.031 0.698 rpy=-1.5708 0 0 -> xyz=0 0.031 0.69 rpy=-1.5708 0 0
- joint r_aj_base: origin xyz=0.0 -0.031 0.698 rpy=1.5708 0 0 -> xyz=0 -0.031 0.69 rpy=1.5708 0 0

File: assets/robot/openarm_tesollo_sensor_rl/openarm_tesollo_sensor_rl.urdf (robot description, URDF)
Before this commit: robot openarm_tesollo_sensor_rl, 53 links, 52 joints
Links:
- added link head_base, mass 0.109629; collision mesh filename=file:///home/user/rl_ws/urdf/vendor/head_realsense_d435i/me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 scale=0.001 0.001 0.001; visual mesh filename=file:///home/user/rl_ws/urdf/vendor/head_realsense_d435i/me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 scale=0.001 0.001 0.001
- added link head_cam_view
- added link head_camera, mass 0.065101; collision mesh filename=file:///home/user/rl_ws/urdf/vendor/head_realsense_d435i/me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 scale=0.001 0.001 0.001; visual mesh filename=file:///home/user/rl_ws/urdf/vendor/head_realsense_d435i/me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 scale=0.001 0.001 0.001
- added link head_mid, mass 0.017073; collision mesh filename=file:///home/user/rl_ws/urdf/vendor/head_realsense_d435i/me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 scale=0.001 0.001 0.001; visual mesh filename=file:///home/user/rl_ws/urdf/vendor/head_realsense_d435i/me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 scale=0.001 0.001 0.001
- link body_link: geometry collision mesh filename=file:///home/user/rl_ws/urdf/generated/rl/meshes/body_link0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 scale=0.001 0.001 0.001; visual mesh filename=file:///home/user/rl_ws/urdf/generated/rl/meshes/body_link0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 scale=0.001 0.001 0.001
Joints:
- added joint head_j_cam_view: type fixed, parent head_camera, child head_cam_view, origin xyz=0.0147 0.0145 0.0365 rpy=0 0 0
- added joint head_j_mount: type fixed, parent body_link, child head_base, origin xyz=0 0 0.750 rpy=0 0 0
- added joint head_j_pan: type revolute, parent head_base, child head_mid, origin xyz=0.0225 0 0.0385 rpy=0 0 0, axis 0 0 -1, limit lower=-1.5708 upper=1.5708 effort=1.0 velocity=6.0
- added joint head_j_tilt: type revolute, parent head_mid, child head_camera, origin xyz=0 -0.0145 0.0275 rpy=0 0 0, axis 0 1 0, limit lower=-1.570796 upper=1.570796 effort=1.0 velocity=6.0
- joint l_aj_base: origin xyz=0.0 0.031 0.698 rpy=-1.5708 0 0 -> xyz=0 0.031 0.69 rpy=-1.5708 0 0
- joint r_aj_base: origin xyz=0.0 -0.031 0.698 rpy=1.5708 0 0 -> xyz=0 -0.031 0.69 rpy=1.5708 0 0
