Commit message: feat(assets): 로봇 자산 재생성분 반영 + openarm_tesollo_bi_s_rl(DG-5FS) 추가
- openarm_tesollo_bi_s_rl 신규(URDF+USD 4종+manifest): DG-5FS 손. 모든 grasp
  태스크가 이 자산으로 전환됨(adf0b24)
- openarm_tesollo_bi_rl / sensor_rl 재생성분: mount 오프셋 0.0595695 → 0.0495
  (-10.07mm) 등 — fabric URDF 재계산(43ae56b)의 근거가 된 변경
- calibration/right_arm.json 삭제: 자산 재생성으로 무효화된 구 실측본.
  소비 코드는 없고 test_calibration_parts 는 부재 시 skip 처리라 안전.
  r2s 재측정 후 재생성 대상
- log_archive/ gitignore 추가 (구 학습 로그 로컬 보관용, 4.5GB)

File: assets/robot/openarm_tesollo_bi_s_rl/openarm_tesollo_bi_s_rl.urdf (robot description, URDF)
Before this commit: robot openarm_dual_tesollo_rl, 84 links, 83 joints
Links:
- link l_hl_adapter: geometry collision mesh filename=file:///home/user/rl_ws/urdf/vendor/delto_m_ros2/dg_descrip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; visual mesh filename=file:///home/user/rl_ws/urdf/vendor/delto_m_ros2/dg_descrip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
- link l_hl_base: mass 0.45 -> 0.11138; geometry collision mesh filename=file:///home/user/rl_ws/urdf/vendor/tesollo_model/dg5fs/mes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; visual mesh filename=file:///home/user/rl_ws/urdf/vendor/tesollo_model/dg5fs/mes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
- link l_hl_index_1: mass 0.045 -> 0.0330237438950368; geometry collision mesh filename=file:///home/user/rl_ws/urdf/vendor/tesollo_model/dg5fs/mes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; visual mesh filename=file:///home/user/rl_ws/urdf/vendor/tesollo_model/dg5fs/mes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
- link l_hl_index_2: mass 0.045 -> 0.0234819993216375; geometry collision mesh filename=file:///home/user/rl_ws/urdf/vendor/tesollo_model/dg5fs/mes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; visual mesh filename=file:///home/user/rl_ws/urdf/vendor/tesollo_model/dg5fs/mes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
- link l_hl_index_3: mass 0.045 -> 0.0234819993216375; geometry collision mesh filename=file:///home/user/rl_ws/urdf/vendor/tesollo_model/dg5fs/mes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; visual mesh filename=file:///home/user/rl_ws/urdf/vendor/tesollo_model/dg5fs/mes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
- link l_hl_index_4: mass 0.025 -> 0.0120970504377428; geometry collision mesh filename=file:///home/user/rl_ws/urdf/vendor/tesollo_model/dg5fs/mes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; visual mesh filename=file:///home/user/rl_ws/urdf/vendor/tesollo_model/dg5fs/mes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
- link l_hl_index_tip: mass 0.005 -> 0.00365660774514008; geometry collision mesh filename=file:///home/user/rl_ws/urdf/vendor/tesollo_model/dg5fs/mes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; visual mesh filename=file:///home/user/rl_ws/urdf/vendor/tesollo_model/dg5fs/mes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
- link l_hl_middle_1: mass 0.045 -> 0.0330237438950368; geometry collision mesh filename=file:///home/user/rl_ws/urdf/vendor/tesollo_model/dg5fs/mes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; visual mesh filename=file:///home/user/rl_ws/urdf/vendor/tesollo_model/dg5fs/mes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
- link l_hl_middle_2: mass 0.045 -> 0.0234819993216375; geometry collision mesh filename=file:///home/user/rl_ws/urdf/vendor/tesollo_model/dg5fs/mes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; visual mesh filename=file:///home/user/rl_ws/urdf/vendor/tesollo_model/dg5fs/mes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
- link l_hl_middle_3: mass 0.045 -> 0.0234819993216375; geometry collision mesh filename=file:///home/user/rl_ws/urdf/vendor/tesollo_model/dg5fs/mes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; visual mesh filename=file:///home/user/rl_ws/urdf/vendor/tesollo_model/dg5fs/mes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
- link l_hl_middle_4: mass 0.025 -> 0.0120970504377428; geometry collision mesh filename=file:///home/user/rl_ws/urdf/vendor/tesollo_model/dg5fs/mes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; visual mesh filename=file:///home/user/rl_ws/urdf/vendor/tesollo_model/dg5fs/mes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
- link l_hl_middle_tip: mass 0.005 -> 0.00365660774513989; geometry collision mesh filename=file:///home/user/rl_ws/urdf/vendor/tesollo_model/dg5fs/mes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; visual mesh filename=file:///home/user/rl_ws/urdf/vendor/tesollo_model/dg5fs/mes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
- link l_hl_palm: mass 0.35 -> 0.520194335203504; geometry collision mesh filename=file:///home/user/rl_ws/urdf/vendor/tesollo_model/dg5fs/mes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; visual mesh filename=file:///home/user/rl_ws/urdf/vendor/tesollo_model/dg5fs/mes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
- link l_hl_pinky_1: mass 0.055 -> 0.0714340581370809; geometry collision mesh filename=file:///home/user/rl_ws/urdf/vendor/tesollo_model/dg5fs/mes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; visual mesh filename=file:///home/user/rl_ws/urdf/vendor/tesollo_model/dg5fs/mes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
- link l_hl_pinky_2: mass 0.025 -> 0.0144987730585103; geometry collision mesh filename=file:///home/user/rl_ws/urdf/vendor/tesollo_model/dg5fs/mes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; visual mesh filename=file:///home/user/rl_ws/urdf/vendor/tesollo_model/dg5fs/mes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
- link l_hl_pinky_3: mass 0.045 -> 0.0234819993216375; geometry collision mesh filename=file:///home/user/rl_ws/urdf/vendor/tesollo_model/dg5fs/mes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; visual mesh filename=file:///home/user/rl_ws/urdf/vendor/tesollo_model/dg5fs/mes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
- link l_hl_pinky_4: mass 0.045 -> 0.0256146776925196; geometry collision mesh filename=file:///home/user/rl_ws/urdf/vendor/tesollo_model/dg5fs/mes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; visual mesh filename=file:///home/user/rl_ws/urdf/vendor/tesollo_model/dg5fs/mes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
- link l_hl_pinky_tip: mass 0.005 -> 0.00365660774514004; geometry collision mesh filename=file:///home/user/rl_ws/urdf/vendor/tesollo_model/dg5fs/mes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; visual mesh filename=file:///home/user/rl_ws/urdf/vendor/tesollo_model/dg5fs/mes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
- link l_hl_ring_1: mass 0.045 -> 0.0330237438950368; geometry collision mesh filename=file:///home/user/rl_ws/urdf/vendor/tesollo_model/dg5fs/mes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; visual mesh filename=file:///home/user/rl_ws/urdf/vendor/tesollo_model/dg5fs/mes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
- link l_hl_ring_2: mass 0.045 -> 0.0234819993216375; geometry collision mesh filename=file:///home/user/rl_ws/urdf/vendor/tesollo_model/dg5fs/mes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; visual mesh filename=file:///home/user/rl_ws/urdf/vendor/tesollo_model/dg5fs/mes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
- link l_hl_ring_3: mass 0.045 -> 0.0234819993216375; geometry collision mesh filename=file:///home/user/rl_ws/urdf/vendor/tesollo_model/dg5fs/mes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; visual mesh filename=file:///home/user/rl_ws/urdf/vendor/tesollo_model/dg5fs/mes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
- link l_hl_ring_4: mass 0.025 -> 0.0120970504377428; geometry collision mesh filename=file:///home/user/rl_ws/urdf/vendor/tesollo_model/dg5fs/mes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; visual mesh filename=file:///home/user/rl_ws/urdf/vendor/tesollo_model/dg5fs/mes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
- link l_hl_ring_tip: mass 0.005 -> 0.00365660774514005; geometry collision mesh filename=file:///home/user/rl_ws/urdf/vendor/tesollo_model/dg5fs/mes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; visual mesh filename=file:///home/user/rl_ws/urdf/vendor/tesollo_model/dg5fs/mes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
- link l_hl_thumb_1: mass 0.045 -> 0.019806363850337; geometry collision mesh filename=file:///home/user/rl_ws/urdf/vendor/tesollo_model/dg5fs/mes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; visual mesh filename=file:///home/user/rl_ws/urdf/vendor/tesollo_model/dg5fs/mes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
- link l_hl_thumb_2: mass 0.025 -> 0.0280995678962355; geometry collision mesh filename=file:///home/user/rl_ws/urdf/vendor/tesollo_model/dg5fs/mes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; visual mesh filename=file:///home/user/rl_ws/urdf/vendor/tesollo_model/dg5fs/mes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
- link l_hl_thumb_3: mass 0.045 -> 0.0234819993216376; geometry collision mesh filename=file:///home/user/rl_ws/urdf/vendor/tesollo_model/dg5fs/mes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; visual mesh filename=file:///home/user/rl_ws/urdf/vendor/tesollo_model/dg5fs/mes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
- link l_hl_thumb_4: mass 0.045 -> 0.0256146769576239; geometry collision mesh filename=file:///home/user/rl_ws/urdf/vendor/tesollo_model/dg5fs/mes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; visual mesh filename=file:///home/user/rl_ws/urdf/vendor/tesollo_model/dg5fs/mes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
- link l_hl_thumb_tip: mass 0.005 -> 0.00365660774514009; geometry collision mesh filename=file:///home/user/rl_ws/urdf/vendor/tesollo_model/dg5fs/mes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; visual mesh filename=file:///home/user/rl_ws/urdf/vendor/tesollo_model/dg5fs/mes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
- link r_hl_adapter: geometry collision mesh filename=file:///home/user/rl_ws/urdf/vendor/delto_m_ros2/dg_descrip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; visual mesh filename=file:///home/user/rl_ws/urdf/vendor/delto_m_ros2/dg_descrip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
- link r_hl_base: mass 0.45 -> 0.11138; geometry collision mesh filename=file:///home/user/rl_ws/urdf/vendor/tesollo_model/dg5fs/mes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; visual mesh filename=file:///home/user/rl_ws/urdf/vendor/tesollo_model/dg5fs/mes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
- link r_hl_index_1: mass 0.045 -> 0.0330237440566374; geometry collision mesh filename=file:///home/user/rl_ws/urdf/vendor/tesollo_model/dg5fs/mes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; visual mesh filename=file:///home/user/rl_ws/urdf/vendor/tesollo_model/dg5fs/mes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
- link r_hl_index_2: mass 0.045 -> 0.0234819993216375; geometry collision mesh filename=file:///home/user/rl_ws/urdf/vendor/tesollo_model/dg5fs/mes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; visual mesh filename=file:///home/user/rl_ws/urdf/vendor/tesollo_model/dg5fs/mes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
- link r_hl_index_3: mass 0.045 -> 0.0234819993216375; geometry collision mesh filename=file:///home/user/rl_ws/urdf/vendor/tesollo_model/dg5fs/mes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; visual mesh filename=file:///home/user/rl_ws/urdf/vendor/tesollo_model/dg5fs/mes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
- link r_hl_index_4: mass 0.025 -> 0.0120970504377428; geometry collision mesh filename=file:///home/user/rl_ws/urdf/vendor/tesollo_model/dg5fs/mes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; visual mesh filename=file:///home/user/rl_ws/urdf/vendor/tesollo_model/dg5fs/mes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
- link r_hl_index_tip: mass 0.005 -> 0.0036566; geometry collision mesh filename=file:///home/user/rl_ws/urdf/vendor/tesollo_model/dg5fs/mes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; visual mesh filename=file:///home/user/rl_ws/urdf/vendor/tesollo_model/dg5fs/mes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
- link r_hl_middle_1: mass 0.045 -> 0.0330237440566374; geometry collision mesh filename=file:///home/user/rl_ws/urdf/vendor/tesollo_model/dg5fs/mes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; visual mesh filename=file:///home/user/rl_ws/urdf/vendor/tesollo_model/dg5fs/mes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
- link r_hl_middle_2: mass 0.045 -> 0.0234819993216375; geometry collision mesh filename=file:///home/user/rl_ws/urdf/vendor/tesollo_model/dg5fs/mes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; visual mesh filename=file:///home/user/rl_ws/urdf/vendor/tesollo_model/dg5fs/mes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
- link r_hl_middle_3: mass 0.045 -> 0.0234819993216375; geometry collision mesh filename=file:///home/user/rl_ws/urdf/vendor/tesollo_model/dg5fs/mes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; visual mesh filename=file:///home/user/rl_ws/urdf/vendor/tesollo_model/dg5fs/mes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
- link r_hl_middle_4: mass 0.025 -> 0.0120970504377428; geometry collision mesh filename=file:///home/user/rl_ws/urdf/vendor/tesollo_model/dg5fs/mes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; visual mesh filename=file:///home/user/rl_ws/urdf/vendor/tesollo_model/dg5fs/mes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
- link r_hl_middle_tip: mass 0.005 -> 0.00365660774514011; geometry collision mesh filename=file:///home/user/rl_ws/urdf/vendor/tesollo_model/dg5fs/mes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; visual mesh filename=file:///home/user/rl_ws/urdf/vendor/tesollo_model/dg5fs/mes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
- link r_hl_palm: mass 0.35 -> 0.52019; geometry collision mesh filename=file:///home/user/rl_ws/urdf/vendor/tesollo_model/dg5fs/mes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; visual mesh filename=file:///home/user/rl_ws/urdf/vendor/tesollo_model/dg5fs/mes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
- link r_hl_pinky_1: mass 0.055 -> 0.0714341385219276; geometry collision mesh filename=file:///home/user/rl_ws/urdf/vendor/tesollo_model/dg5fs/mes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; visual mesh filename=file:///home/user/rl_ws/urdf/vendor/tesollo_model/dg5fs/mes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
- link r_hl_pinky_2: mass 0.025 -> 0.0144987730585103; geometry collision mesh filename=file:///home/user/rl_ws/urdf/vendor/tesollo_model/dg5fs/mes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; visual mesh filename=file:///home/user/rl_ws/urdf/vendor/tesollo_model/dg5fs/mes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
- link r_hl_pinky_3: mass 0.045 -> 0.0234819993216375; geometry collision mesh filename=file:///home/user/rl_ws/urdf/vendor/tesollo_model/dg5fs/mes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; visual mesh filename=file:///home/user/rl_ws/urdf/vendor/tesollo_model/dg5fs/mes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
- link r_hl_pinky_4: mass 0.045 -> 0.0256146776925196; geometry collision mesh filename=file:///home/user/rl_ws/urdf/vendor/tesollo_model/dg5fs/mes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; visual mesh filename=file:///home/user/rl_ws/urdf/vendor/tesollo_model/dg5fs/mes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
- link r_hl_pinky_tip: mass 0.005 -> 0.00365660774514004; geometry collision mesh filename=file:///home/user/rl_ws/urdf/vendor/tesollo_model/dg5fs/mes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; visual mesh filename=file:///home/user/rl_ws/urdf/vendor/tesollo_model/dg5fs/mes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
- link r_hl_ring_1: mass 0.045 -> 0.0330237440566374; geometry collision mesh filename=file:///home/user/rl_ws/urdf/vendor/tesollo_model/dg5fs/mes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; visual mesh filename=file:///home/user/rl_ws/urdf/vendor/tesollo_model/dg5fs/mes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
- link r_hl_ring_2: mass 0.045 -> 0.0234819976154512; geometry collision mesh filename=file:///home/user/rl_ws/urdf/vendor/tesollo_model/dg5fs/mes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; visual mesh filename=file:///home/user/rl_ws/urdf/vendor/tesollo_model/dg5fs/mes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
- link r_hl_ring_3: mass 0.045 -> 0.0234819993216375; geometry collision mesh filename=file:///home/user/rl_ws/urdf/vendor/tesollo_model/dg5fs/mes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; visual mesh filename=file:///home/user/rl_ws/urdf/vendor/tesollo_model/dg5fs/mes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
- link r_hl_ring_4: mass 0.025 -> 0.0120970504377428; geometry collision mesh filename=file:///home/user/rl_ws/urdf/vendor/tesollo_model/dg5fs/mes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; visual mesh filename=file:///home/user/rl_ws/urdf/vendor/tesollo_model/dg5fs/mes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
- link r_hl_ring_tip: mass 0.005 -> 0.0036566077451401; geometry collision mesh filename=file:///home/user/rl_ws/urdf/vendor/tesollo_model/dg5fs/mes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; visual mesh filename=file:///home/user/rl_ws/urdf/vendor/tesollo_model/dg5fs/mes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
- link r_hl_thumb_1: mass 0.045 -> 0.0198063638503371; geometry collision mesh filename=file:///home/user/rl_ws/urdf/vendor/tesollo_model/dg5fs/mes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; visual mesh filename=file:///home/user/rl_ws/urdf/vendor/tesollo_model/dg5fs/mes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
- link r_hl_thumb_2: mass 0.025 -> 0.0280995687846082; geometry collision mesh filename=file:///home/user/rl_ws/urdf/vendor/tesollo_model/dg5fs/mes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; visual mesh filename=file:///home/user/rl_ws/urdf/vendor/tesollo_model/dg5fs/mes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
- link r_hl_thumb_3: mass 0.045 -> 0.0234819983656458; geometry collision mesh filename=file:///home/user/rl_ws/urdf/vendor/tesollo_model/dg5fs/mes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; visual mesh filename=file:///home/user/rl_ws/urdf/vendor/tesollo_model/dg5fs/mes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
- link r_hl_thumb_4: mass 0.045 -> 0.0256150236808272; geometry collision mesh filename=file:///home/user/rl_ws/urdf/vendor/tesollo_model/dg5fs/mes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; visual mesh filename=file:///home/user/rl_ws/urdf/vendor/tesollo_model/dg5fs/mes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
- link r_hl_thumb_tip: mass 0.005 -> 0.00365660774514007; geometry collision mesh filename=file:///home/user/rl_ws/urdf/vendor/tesollo_model/dg5fs/mes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; visual mesh filename=file:///home/user/rl_ws/urdf/vendor/tesollo_model/dg5fs/mes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
Joints:
- joint l_hj_index_1: axis 1 0 0 -> 0 0 1; limit lower=-0.6108652381980153 upper=0.4188790204786391 effort=7.5 velocity=3.141592653589793 -> lower=-0.2617993877991494 upper=0.8377580409572782 effort=7.5 velocity=3.141592653589793; origin xyz=-0.0071 -0.027 0.0661 rpy=0.0 0.0 0.0 -> xyz=0.0017 -0.028 0.08365 rpy=3.1416 -1.5708 0
- joint l_hj_index_2: axis 0 1 0 -> 0 0 1; limit lower=-0.0 upper=2.007128639793479 effort=7.5 velocity=3.141592653589793 -> lower=0 upper=2.199114857512855 effort=7.5 velocity=3.141592653589793; origin xyz=0.01765 0.0 0.0265 rpy=0.0 0.0 0.0 -> xyz=0.02415 0 0.0126 rpy=1.5708 0 0
- joint l_hj_index_3: axis 0 1 0 -> 0 0 1; origin xyz=0.0 0.0 0.0388 rpy=0.0 0.0 0.0 -> xyz=0.0334 0 0 rpy=0 0 0
- joint l_hj_index_4: axis 0 1 0 -> 0 0 1; origin xyz=0.0 0.0 0.0388 rpy=0.0 0.0 0.0 -> xyz=0.0334 0 0 rpy=0 0 0
- joint l_hj_index_tip: axis (none) -> 0 0 0; origin xyz=0.0 0.0 0.0255 rpy=0.0 0.0 0.0 -> xyz=0.018 0 0 rpy=0 0 0
- joint l_hj_middle_1: axis 1 0 0 -> 0 0 1; limit lower=-0.6108652381980153 upper=0.6108652381980153 effort=7.5 velocity=3.141592653589793 -> lower=-0.7330382858376184 upper=0.5759586531581288 effort=7.5 velocity=3.141592653589793; origin xyz=-0.0071 -0.0025 0.0701 rpy=0.0 0.0 0.0 -> xyz=0.0017 -0.005 0.08865 rpy=3.1416 -1.5708 0
- joint l_hj_middle_2: axis 0 1 0 -> 0 0 1; limit lower=-0.0 upper=1.9547687622336491 effort=7.5 velocity=3.141592653589793 -> lower=0 upper=2.2689280275926285 effort=7.5 velocity=3.141592653589793; origin xyz=0.01765 0.0 0.0265 rpy=0.0 0.0 0.0 -> xyz=0.02415 0 0.0126 rpy=1.5708 0 0
- joint l_hj_middle_3: axis 0 1 0 -> 0 0 1; origin xyz=0.0 0.0 0.0388 rpy=0.0 0.0 0.0 -> xyz=0.0334 0 0 rpy=0 0 0
- joint l_hj_middle_4: axis 0 1 0 -> 0 0 1; origin xyz=0.0 0.0 0.0388 rpy=0.0 0.0 0.0 -> xyz=0.0334 0 0 rpy=0 0 0
- joint l_hj_middle_tip: axis (none) -> 0 0 0; origin xyz=0.0 0.0 0.0255 rpy=0.0 0.0 0.0 -> xyz=0.018 0 0 rpy=0 0 0
- joint l_hj_palm: axis (none) -> 0 0 0; origin xyz=0 0 0.0698 rpy=0 0 0 -> xyz=0 0 0.015 rpy=0 0 0
- joint l_hj_pinky_1: limit lower=-1.0471975511965976 upper=0.017453292519943295 effort=7.5 velocity=3.141592653589793 -> lower=-1.0471975511965976 upper=0 effort=7.5 velocity=3.141592653589793; origin xyz=0.0103 0.0195 0.0182 rpy=0.0 0.0 0.0 -> xyz=0.013 0.01805 0.0364 rpy=0 0 1.5708
- joint l_hj_pinky_2: axis 1 0 0 -> 0 0 1; limit lower=-0.6108652381980153 upper=0.4188790204786391 effort=7.5 velocity=3.141592653589793 -> lower=-1.5707963267948966 upper=0.6457718232379019 effort=7.5 velocity=3.141592653589793; origin xyz=0.0 0.028 0.0381 rpy=0.0 0.0 0.0 -> xyz=0.02445 0 0.0307 rpy=1.5708 0 0
- joint l_hj_pinky_3: axis 0 1 0 -> 0 0 1; origin xyz=0.0 0.0 0.031 rpy=0.0 0.0 0.0 -> xyz=0 0.0272 0 rpy=1.5708 0 1.5708
- joint l_hj_pinky_4: axis 0 1 0 -> 0 0 1; origin xyz=0.0 0.0 0.0388 rpy=0.0 0.0 0.0 -> xyz=0.0334 0 0 rpy=0 0 0
- joint l_hj_pinky_tip: axis (none) -> 0 0 0; origin xyz=0.0 0.0 0.0363 rpy=0.0 0.0 0.0 -> xyz=0.0289 0 0 rpy=0 0 0
- joint l_hj_ring_1: axis 1 0 0 -> 0 0 1; limit lower=-0.4188790204786391 upper=0.6108652381980153 effort=7.5 velocity=3.141592653589793 -> lower=-0.8377580409572782 upper=0.20943951023931956 effort=7.5 velocity=3.141592653589793; origin xyz=-0.0071 0.022 0.0621 rpy=0.0 0.0 0.0 -> xyz=0.0017 0.018 0.08065 rpy=3.1416 -1.5708 0
- joint l_hj_ring_2: axis 0 1 0 -> 0 0 1; limit lower=-0.0 upper=1.9024088846738192 effort=7.5 velocity=3.141592653589793 -> lower=0 upper=2.2165681500327987 effort=7.5 velocity=3.141592653589793; origin xyz=0.01765 0.0 0.0265 rpy=0.0 0.0 0.0 -> xyz=0.02415 0 0.0126 rpy=1.5708 0 0
- joint l_hj_ring_3: axis 0 1 0 -> 0 0 1; origin xyz=0.0 0.0 0.0388 rpy=0.0 0.0 0.0 -> xyz=0.0334 0 0 rpy=0 0 0
- joint l_hj_ring_4: axis 0 1 0 -> 0 0 1; origin xyz=0.0 0.0 0.0388 rpy=0.0 0.0 0.0 -> xyz=0.0334 0 0 rpy=0 0 0
- joint l_hj_ring_tip: axis (none) -> 0 0 0; origin xyz=0.0 0.0 0.0255 rpy=0.0 0.0 0.0 -> xyz=0.018 0 0 rpy=0 0 0
- joint l_hj_thumb_1: axis 1 0 0 -> 0 0 1; limit lower=-0.8901179185171081 upper=0.3839724354387525 effort=7.5 velocity=3.141592653589793 -> lower=-1.5707963267948966 upper=1.5707963267948966 effort=7.5 velocity=3.141592653589793; origin xyz=-0.0162 -0.019 0.0128 rpy=0.0 0.0 0.0 -> xyz=0.0017 -0.018 0.0298 rpy=-1.5708 0 -1.5708
- joint l_hj_thumb_2: limit lower=-0.0 upper=3.141592653589793 effort=7.5 velocity=3.141592653589793 -> lower=0 upper=2.670353755551324 effort=7.5 velocity=3.141592653589793; origin xyz=0.04195 0.0 0.0 rpy=0.0 0.0 0.0 -> xyz=0 0 0.0262 rpy=1.5708 0 0
- joint l_hj_thumb_3: axis 1 0 0 -> 0 0 1; origin xyz=0.0 -0.031 0.0 rpy=0.0 0.0 0.0 -> xyz=0.0381 0 0 rpy=-1.5708 0 0
- joint l_hj_thumb_4: axis 1 0 0 -> 0 0 1; origin xyz=0.0 -0.0388 0.0 rpy=0.0 0.0 0.0 -> xyz=0.0334 0 0 rpy=0 0 0
- joint l_hj_thumb_tip: axis (none) -> 0 0 0; origin xyz=0.0 -0.0363 0.0 rpy=0.0 0.0 0.0 -> xyz=0.0289 0 0 rpy=0 0 0
- joint r_hj_index_1: axis 1 0 0 -> 0 0 1; limit lower=-0.4188790204786391 upper=0.6108652381980153 effort=7.5 velocity=3.141592653589793 -> lower=-0.8377580409572782 upper=0.2617993877991494 effort=7.5 velocity=3.141592653589793; origin xyz=-0.0071 0.027 0.0661 rpy=0.0 0.0 0.0 -> xyz=0.0017 0.028 0.08365 rpy=3.1416 -1.5708 0
- joint r_hj_index_2: axis 0 1 0 -> 0 0 -1; limit lower=-0.0 upper=2.007128639793479 effort=7.5 velocity=3.141592653589793 -> lower=0 upper=2.199114857512855 effort=7.5 velocity=3.141592653589793; origin xyz=0.01765 0.0 0.0265 rpy=0.0 0.0 0.0 -> xyz=0.02415 0 0.0126 rpy=-1.5708 0 0
- joint r_hj_index_3: axis 0 1 0 -> 0 0 1; origin xyz=0.0 0.0 0.0388 rpy=0.0 0.0 0.0 -> xyz=0.0334 0 0 rpy=3.1416 0 0
- joint r_hj_index_4: axis 0 1 0 -> 0 0 1; origin xyz=0.0 0.0 0.0388 rpy=0.0 0.0 0.0 -> xyz=0.0334 0 0 rpy=0 0 0
- joint r_hj_index_tip: axis (none) -> 0 0 0; origin xyz=0.0 0.0 0.0255 rpy=0.0 0.0 0.0 -> xyz=0.018 0 0 rpy=0 0 0
- joint r_hj_middle_1: axis 1 0 0 -> 0 0 1; limit lower=-0.6108652381980153 upper=0.6108652381980153 effort=7.5 velocity=3.141592653589793 -> lower=-0.5759586531581288 upper=0.7330382858376184 effort=7.5 velocity=3.141592653589793; origin xyz=-0.0071 0.0025 0.0701 rpy=0.0 0.0 0.0 -> xyz=0.0017 0.005 0.08865 rpy=3.1416 -1.5708 0
- joint r_hj_middle_2: axis 0 1 0 -> 0 0 -1; limit lower=-0.0 upper=1.9547687622336491 effort=7.5 velocity=3.141592653589793 -> lower=0 upper=2.2689280275926285 effort=7.5 velocity=3.141592653589793; origin xyz=0.01765 0.0 0.0265 rpy=0.0 0.0 0.0 -> xyz=0.02415 0 0.0126 rpy=-1.5708 0 0
- joint r_hj_middle_3: axis 0 1 0 -> 0 0 1; origin xyz=0.0 0.0 0.0388 rpy=0.0 0.0 0.0 -> xyz=0.0334 0 0 rpy=3.1416 0 0
- joint r_hj_middle_4: axis 0 1 0 -> 0 0 1; origin xyz=0.0 0.0 0.0388 rpy=0.0 0.0 0.0 -> xyz=0.0334 0 0 rpy=0 0 0
- joint r_hj_middle_tip: axis (none) -> 0 0 0; origin xyz=0.0 0.0 0.0255 rpy=0.0 0.0 0.0 -> xyz=0.018 0 0 rpy=0 0 0
- joint r_hj_palm: axis (none) -> 0 0 0; origin xyz=0 0 0.0698 rpy=0 0 0 -> xyz=0 0 0.015 rpy=0 0 0
- joint r_hj_pinky_1: limit lower=-0.017453292519943295 upper=1.0471975511965976 effort=7.5 velocity=3.141592653589793 -> lower=0 upper=1.0471975511965976 effort=7.5 velocity=3.141592653589793; origin xyz=0.0103 -0.0195 0.0182 rpy=0.0 0.0 0.0 -> xyz=0.013 -0.01805 0.0364 rpy=0 0 -1.5708
- joint r_hj_pinky_2: axis 1 0 0 -> 0 0 1; limit lower=-0.4188790204786391 upper=0.6108652381980153 effort=7.5 velocity=3.141592653589793 -> lower=-0.6457718232379019 upper=1.5707963267948966 effort=7.5 velocity=3.141592653589793; origin xyz=0.0 -0.028 0.0381 rpy=0.0 0.0 0.0 -> xyz=0.02445 0 0.0307 rpy=-1.5708 0 0
- joint r_hj_pinky_3: axis 0 1 0 -> 0 0 1; origin xyz=0.0 0.0 0.031 rpy=0.0 0.0 0.0 -> xyz=0 -0.0272 0 rpy=1.5708 0 -1.5708
- joint r_hj_pinky_4: axis 0 1 0 -> 0 0 1; origin xyz=0.0 0.0 0.0388 rpy=0.0 0.0 0.0 -> xyz=0.0334 0 0 rpy=0 0 0
- joint r_hj_pinky_tip: axis (none) -> 0 0 0; origin xyz=0.0 0.0 0.0363 rpy=0.0 0.0 0.0 -> xyz=0.0289 0 0 rpy=0 0 0
- joint r_hj_ring_1: axis 1 0 0 -> 0 0 1; limit lower=-0.6108652381980153 upper=0.4188790204786391 effort=7.5 velocity=3.141592653589793 -> lower=-0.20943951023931956 upper=0.8377580409572782 effort=7.5 velocity=3.141592653589793; origin xyz=-0.0071 -0.022 0.0621 rpy=0.0 0.0 0.0 -> xyz=0.0013 -0.018 0.08065 rpy=3.1416 -1.5708 0
- joint r_hj_ring_2: axis 0 1 0 -> 0 0 -1; limit lower=-0.0 upper=1.9024088846738192 effort=7.5 velocity=3.141592653589793 -> lower=0 upper=2.2165681500327987 effort=7.5 velocity=3.141592653589793; origin xyz=0.01765 0.0 0.0265 rpy=0.0 0.0 0.0 -> xyz=0.02415 0 0.0126 rpy=-1.5708 0 0
- joint r_hj_ring_3: axis 0 1 0 -> 0 0 1; origin xyz=0.0 0.0 0.0388 rpy=0.0 0.0 0.0 -> xyz=0.0334 0 0 rpy=3.1416 0 0
- joint r_hj_ring_4: axis 0 1 0 -> 0 0 1; origin xyz=0.0 0.0 0.0388 rpy=0.0 0.0 0.0 -> xyz=0.0334 0 0 rpy=0 0 0
- joint r_hj_ring_tip: axis (none) -> 0 0 0; origin xyz=0.0 0.0 0.0255 rpy=0.0 0.0 0.0 -> xyz=0.018 0 0 rpy=0 0 0
- joint r_hj_thumb_1: axis 1 0 0 -> 0 0 1; limit lower=-0.3839724354387525 upper=0.8901179185171081 effort=7.5 velocity=3.141592653589793 -> lower=-1.5707963267948966 upper=1.5707963267948966 effort=7.5 velocity=3.141592653589793; origin xyz=-0.0162 0.019 0.0128 rpy=0.0 0.0 0.0 -> xyz=0.0017 0.018 0.0298 rpy=1.5708 0 1.5708
- joint r_hj_thumb_2: limit lower=-3.141592653589793 upper=0.0 effort=7.5 velocity=3.141592653589793 -> lower=-2.670353755551324 upper=0 effort=7.5 velocity=3.141592653589793; origin xyz=0.04195 0.0 0.0 rpy=0.0 0.0 0.0 -> xyz=0 0 0.0262 rpy=-1.5708 0 0
- joint r_hj_thumb_3: axis 1 0 0 -> 0 0 1; origin xyz=0.0 0.031 0.0 rpy=0.0 0.0 0.0 -> xyz=0.0381 0 0 rpy=1.5708 0 0
- joint r_hj_thumb_4: axis 1 0 0 -> 0 0 1; origin xyz=0.0 0.0388 0.0 rpy=0.0 0.0 0.0 -> xyz=0.0334 0 0 rpy=0 0 0
- joint r_hj_thumb_tip: axis (none) -> 0 0 0; origin xyz=0.0 0.0363 0.0 rpy=0.0 0.0 0.0 -> xyz=0.0289 0 0 rpy=0 0 0
