Commit message: fix(assets): 로봇 자산 4종 재빌드 — head_v1 RGB 렌즈 개구부 정정(hand-eye v2) + USD 에 head_v1.usda 직접 이식
- head_cam_view / manifest camera_view_frame 을 head_v1 의 y+0.0326 개구부(ir_projector_frame 라벨)로 이동: CAD 사전 모델
  hand-eye 재계산 RMS 1.86 px(color_frame 5.94), 테이블 0.204(줄자 0.205), 홈 실사진 vs sim 렌더 일치.
- USD 의 head 지오메트리는 head_v1.usda 참조(머티리얼·광학 프레임 프림 보존, 참조 physics 제거). 카메라는
  <root>/head_camera/head_v1/camera_link/ir_projector_frame 에 붙이면 실기 RGB 자리다.
- 무질량 프레임·RH56F1 벤더 0 질량 링크 1e-5 kg, DG-5F 손 1.763 kg, body 하우징 제거, 벤더 게인.

Co-Authored-By: Claude Fable 5.1 <noreply@anthropic.com>
Claude-Session: https://claude.ai/code/session_01B2gFUoGNzc6ZVktHojTXc7

File: assets/robot/openarm_dg5f-m_bi_rl/openarm_dg5f-m_bi_rl.urdf (robot description, URDF)
Before this commit: robot openarm_dg5f_m_bi_rl, 84 links, 83 joints
Joints:
- joint head_j_cam_view: origin xyz=0.0115 9.6e-05 0.036327 rpy=0 0 0 -> xyz=0.01236 0.044096 0.036317 rpy=0 0 0

File: assets/robot/openarm_dg5f-s_bi_rl/openarm_dg5f-s_bi_rl.urdf (robot description, URDF)
Before this commit: robot openarm_dg5f_s_bi_rl, 84 links, 83 joints
Joints:
- joint head_j_cam_view: origin xyz=0.0115 9.6e-05 0.036327 rpy=0 0 0 -> xyz=0.01236 0.044096 0.036317 rpy=0 0 0

File: assets/robot/openarm_gripper_bi_rl/openarm_gripper_bi_rl.urdf (robot description, URDF)
Before this commit: robot openarm_gripper_bi_rl, 30 links, 29 joints
Joints:
- joint head_j_cam_view: origin xyz=0.0115 9.6e-05 0.036327 rpy=0 0 0 -> xyz=0.01236 0.044096 0.036317 rpy=0 0 0

File: assets/robot/openarm_rh56f1_bi_rl/openarm_rh56f1_bi_rl.urdf (robot description, URDF)
Before this commit: robot openarm_rh56f1_bi_rl, 76 links, 75 joints
Joints:
- joint head_j_cam_view: origin xyz=0.0115 9.6e-05 0.036327 rpy=0 0 0 -> xyz=0.01236 0.044096 0.036317 rpy=0 0 0
