Commit message: fix(fabric): short 자산 어댑터 삽입 반영 — fabric URDF 재생성 + 구 패치 재적용
988a2186 이 short 자산에 플랜지 어댑터(10mm)를 삽입해 palm 이 옮겨졌는데 fabric URDF 는
그 이전 값을 들고 있었다. 부팅 게이트가 잡았다:

  RuntimeError: [tesollo_right_short] fabric FK 가 USD palm 과 어긋난다: 9.8mm / 0.2°

9.8mm 는 어댑터 10mm 와 일치한다. 재생성 후 **1.86mm / 0.23°** (허용 5mm/2°).

★파이프라인이 2단계라는 것을 이번에 확정했다:
    gen_fabric_urdfs.py <variant> --sync-hdgp     → 기본 62 링크
    patch_fabric_finger_spheres.py --robot … --params …  → 손가락 구 52개 → 104 링크
  생성기가 실행 끝에 이 후처리 명령줄을 그대로 출력하는데, **그 NOTE 는 `--sync-hdgp`
  분기에서만 찍힌다.** 오전에 조사하며 sync 를 빼고 돌렸다가 그 안내를 놓쳤고,
  "재생성은 구 레이아웃(62 링크 _sphere*)을 내므로 오답"이라고 잘못 결론냈다.
  실제로는 재생성이 맞고 후처리를 빠뜨린 것이었다. 조사용 dry 실행은 부작용과 함께
  **안내문도** 건너뛴다.

★후처리 스크립트에 멱등성 가드가 없다. 두 번 돌면 링크가 104 → 156 으로 늘고
  urdfpy 가 중복 이름으로 로드를 거부한다(dcb0b0c3 에서 그 상태를 수동 정리했다).
  재생성으로 62 기준선을 만든 뒤 **정확히 한 번씩만** 돌릴 것.

검증: 좌우 각 link 104(고유 104) · joint 103(고유 103) · 동작본 openarm_dg5f-m_bi_right 와
  링크명 집합 차이 0. params 도 _sph 고유 52 · 중복 키 0 · 동작본과 집합차 0.
  부팅: obs=140 state=158 action=21 · fabric=openarm_dg5f-m-short_bi_right · FK 1.86mm

Co-Authored-By: Claude Opus 5 <noreply@anthropic.com>
Claude-Session: https://claude.ai/code/session_01HvcDZwv5KQCbEQfov6g9Vb

File: source/FABRICS/src/fabrics_sim/models/robots/urdf/openarm_dg5f-m-short_bi_left/openarm_dg5f-m-short_bi_left.urdf (robot description, URDF)
Before this commit: robot openarm_dg5f-m-short_bi_left, 104 links, 103 joints
Links:
- link palm_link: mass 0.75723 -> 0.75721
Joints:
- joint palm_link_joint: origin xyz=0 -3e-07 0.076 rpy=0 0 1.5707964 -> xyz=0 -3e-07 0.086 rpy=0 0 1.5707964
- joint rj_dg_1_1: limit lower=-1.34390352 upper=0.383972435 effort=7.5 velocity=3.1415927 -> lower=-1.3439 upper=0.383972 effort=7.5 velocity=3.1415927
- joint rj_dg_1_2: limit lower=-0 upper=2.70526034 effort=7.5 velocity=3.1415927 -> lower=-0 upper=2.70526 effort=7.5 velocity=3.1415927
- joint rj_dg_1_3: limit lower=-1.57079633 upper=1.57079633 effort=7.5 velocity=3.1415927 -> lower=-1.5708 upper=1.5708 effort=7.5 velocity=3.1415927
- joint rj_dg_1_4: limit lower=-1.57079633 upper=1.57079633 effort=7.5 velocity=3.1415927 -> lower=-1.5708 upper=1.5708 effort=7.5 velocity=3.1415927
- joint rj_dg_2_1: limit lower=-0.34906585 upper=0.541052068 effort=7.5 velocity=3.1415927 -> lower=-0.349066 upper=0.541052 effort=7.5 velocity=3.1415927
- joint rj_dg_2_2: limit lower=-0 upper=2.00712864 effort=7.5 velocity=3.1415927 -> lower=0 upper=2.00713 effort=7.5 velocity=3.1415927
- joint rj_dg_2_3: limit lower=-1.57079633 upper=1.57079633 effort=7.5 velocity=3.1415927 -> lower=-1.5708 upper=1.5708 effort=7.5 velocity=3.1415927
- joint rj_dg_2_4: limit lower=-1.57079633 upper=1.57079633 effort=7.5 velocity=3.1415927 -> lower=-1.5708 upper=1.5708 effort=7.5 velocity=3.1415927
- joint rj_dg_3_1: limit lower=-0.436332313 upper=0.436332313 effort=7.5 velocity=3.1415927 -> lower=-0.436332 upper=0.436332 effort=7.5 velocity=3.1415927
- joint rj_dg_3_2: limit lower=0 upper=2.00712864 effort=7.5 velocity=3.1415927 -> lower=0 upper=2.00713 effort=7.5 velocity=3.1415927
- joint rj_dg_3_3: limit lower=-1.57079633 upper=1.57079633 effort=7.5 velocity=3.1415927 -> lower=-1.5708 upper=1.5708 effort=7.5 velocity=3.1415927
- joint rj_dg_3_4: limit lower=-1.57079633 upper=1.57079633 effort=7.5 velocity=3.1415927 -> lower=-1.5708 upper=1.5708 effort=7.5 velocity=3.1415927
- joint rj_dg_4_1: limit lower=-0.558505361 upper=0.261799388 effort=7.5 velocity=3.1415927 -> lower=-0.558505 upper=0.261799 effort=7.5 velocity=3.1415927
- joint rj_dg_4_2: limit lower=0 upper=1.91986218 effort=7.5 velocity=3.1415927 -> lower=0 upper=1.91986 effort=7.5 velocity=3.1415927
- joint rj_dg_4_3: limit lower=-1.57079633 upper=1.57079633 effort=7.5 velocity=3.1415927 -> lower=-1.5708 upper=1.5708 effort=7.5 velocity=3.1415927
- joint rj_dg_4_4: limit lower=-1.57079633 upper=1.57079633 effort=7.5 velocity=3.1415927 -> lower=-1.5708 upper=1.5708 effort=7.5 velocity=3.1415927
- joint rj_dg_5_1: limit lower=-1.04719755 upper=0 effort=7.5 velocity=3.1415927 -> lower=-1.0472 upper=-0 effort=7.5 velocity=3.1415927
- joint rj_dg_5_2: limit lower=-1.57079633 upper=0.261799388 effort=7.5 velocity=3.1415927 -> lower=-1.5708 upper=0.261799 effort=7.5 velocity=3.1415927
- joint rj_dg_5_3: limit lower=-1.57079633 upper=1.57079633 effort=7.5 velocity=3.1415927 -> lower=-1.5708 upper=1.5708 effort=7.5 velocity=3.1415927
- joint rj_dg_5_4: limit lower=-1.57079633 upper=1.57079633 effort=7.5 velocity=3.1415927 -> lower=-1.5708 upper=1.5708 effort=7.5 velocity=3.1415927

File: source/FABRICS/src/fabrics_sim/models/robots/urdf/openarm_dg5f-m-short_bi_right/openarm_dg5f-m-short_bi_right.urdf (robot description, URDF)
Before this commit: robot openarm_dg5f-m-short_bi_right, 104 links, 103 joints
Links:
- link palm_link: mass 0.75723 -> 0.75721
Joints:
- joint palm_link_joint: origin xyz=0 3e-07 0.076 rpy=0. 0. -1.5707964 -> xyz=0 3e-07 0.086 rpy=0. 0. -1.5707964
- joint rj_dg_1_1: limit lower=-0.383972435 upper=1.34390352 effort=7.5 velocity=3.1415927 -> lower=-0.383972 upper=1.3439 effort=7.5 velocity=3.1415927
- joint rj_dg_1_2: limit lower=-2.70526034 upper=0 effort=7.5 velocity=3.1415927 -> lower=-2.70526 upper=0 effort=7.5 velocity=3.1415927
- joint rj_dg_1_3: limit lower=-1.57079633 upper=1.57079633 effort=7.5 velocity=3.1415927 -> lower=-1.5708 upper=1.5708 effort=7.5 velocity=3.1415927
- joint rj_dg_1_4: limit lower=-1.57079633 upper=1.57079633 effort=7.5 velocity=3.1415927 -> lower=-1.5708 upper=1.5708 effort=7.5 velocity=3.1415927
- joint rj_dg_2_1: limit lower=-0.541052068 upper=0.34906585 effort=7.5 velocity=3.1415927 -> lower=-0.541052 upper=0.349066 effort=7.5 velocity=3.1415927
- joint rj_dg_2_2: limit lower=-0 upper=2.00712864 effort=7.5 velocity=3.1415927 -> lower=0 upper=2.00713 effort=7.5 velocity=3.1415927
- joint rj_dg_2_3: limit lower=-1.57079633 upper=1.57079633 effort=7.5 velocity=3.1415927 -> lower=-1.5708 upper=1.5708 effort=7.5 velocity=3.1415927
- joint rj_dg_2_4: limit lower=-1.57079633 upper=1.57079633 effort=7.5 velocity=3.1415927 -> lower=-1.5708 upper=1.5708 effort=7.5 velocity=3.1415927
- joint rj_dg_3_1: limit lower=-0.436332313 upper=0.436332313 effort=7.5 velocity=3.1415927 -> lower=-0.436332 upper=0.436332 effort=7.5 velocity=3.1415927
- joint rj_dg_3_2: limit lower=0 upper=2.00712864 effort=7.5 velocity=3.1415927 -> lower=0 upper=2.00713 effort=7.5 velocity=3.1415927
- joint rj_dg_3_3: limit lower=-1.57079633 upper=1.57079633 effort=7.5 velocity=3.1415927 -> lower=-1.5708 upper=1.5708 effort=7.5 velocity=3.1415927
- joint rj_dg_3_4: limit lower=-1.57079633 upper=1.57079633 effort=7.5 velocity=3.1415927 -> lower=-1.5708 upper=1.5708 effort=7.5 velocity=3.1415927
- joint rj_dg_4_1: limit lower=-0.261799388 upper=0.558505361 effort=7.5 velocity=3.1415927 -> lower=-0.261799 upper=0.558505 effort=7.5 velocity=3.1415927
- joint rj_dg_4_2: limit lower=0 upper=1.91986218 effort=7.5 velocity=3.1415927 -> lower=0 upper=1.91986 effort=7.5 velocity=3.1415927
- joint rj_dg_4_3: limit lower=-1.57079633 upper=1.57079633 effort=7.5 velocity=3.1415927 -> lower=-1.5708 upper=1.5708 effort=7.5 velocity=3.1415927
- joint rj_dg_4_4: limit lower=-1.57079633 upper=1.57079633 effort=7.5 velocity=3.1415927 -> lower=-1.5708 upper=1.5708 effort=7.5 velocity=3.1415927
- joint rj_dg_5_1: limit lower=-0 upper=1.04719755 effort=7.5 velocity=3.1415927 -> lower=0 upper=1.0472 effort=7.5 velocity=3.1415927
- joint rj_dg_5_2: limit lower=-0.261799388 upper=1.57079633 effort=7.5 velocity=3.1415927 -> lower=-0.261799 upper=1.5708 effort=7.5 velocity=3.1415927
- joint rj_dg_5_3: limit lower=-1.57079633 upper=1.57079633 effort=7.5 velocity=3.1415927 -> lower=-1.5708 upper=1.5708 effort=7.5 velocity=3.1415927
- joint rj_dg_5_4: limit lower=-1.57079633 upper=1.57079633 effort=7.5 velocity=3.1415927 -> lower=-1.5708 upper=1.5708 effort=7.5 velocity=3.1415927
