Commit message: fix(assets): RH56F1 자산 재빌드 — 전 링크 convex hull·자기충돌 필터 54·손 드라이브 30/0.3·mimic nf 500
rl_ws/urdf tools/build_usd.py openarm_rh56f1_bi_rl --sync-hdgp (RH56F1 폴더만).
사용자 09.15: dg5f-m-short 처럼 전체 convex hull, 자기충돌 ON 에서도 링크 간 충돌 없음, 손가락 흔들림(액추에이터) 정정.
- colliders 75 전부 convexHull(손 54, 벤더 STL · primitive·palm_1 제거 폐지), 필터 54 body pair
  (zero + 손 자세 4종 감사 PASS, 손바닥↔손가락 원위·엄지↔손가락 필터 없음)
- 손 구동 12관절 드라이브 30 N·m/rad / 0.3 (fallback 100/1 폐지), mimic 12쌍 naturalFrequency 500
- 근거: probes/probe_rh56f1_finger_sweep.py 실측(메모리 rh56f1-finger-shake-actuator-probe)
- ★hdgp 학습 게인(robot_profiles RH56F1 hand 5/2)은 spawn 에서 덮어쓴다 — 변경은 사용자 결정 대기

Co-Authored-By: Claude Opus 5 <noreply@anthropic.com>
Claude-Session: https://claude.ai/code/session_016RobHoZyV19R1xziMustBN

File: assets/robot/openarm_rh56f1_bi_rl/openarm_rh56f1_bi_rl.urdf (robot description, URDF)
Before this commit: robot openarm_rh56f1_bi_rl, 76 links, 75 joints
Links:
- link l_hl_index_1: geometry collision mesh filename=file:///home/user/rl_ws/urdf/vendor/RH56F1/RH56F1_L/meshes/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; visual mesh filename=file:///home/user/rl_ws/urdf/vendor/RH56F1/RH56F1_L/meshes/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
- link l_hl_index_2: geometry collision mesh filename=file:///home/user/rl_ws/urdf/vendor/RH56F1/RH56F1_L/meshes/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; visual mesh filename=file:///home/user/rl_ws/urdf/vendor/RH56F1/RH56F1_L/meshes/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
- link l_hl_index_sensor: geometry collision mesh filename=file:///home/user/rl_ws/urdf/vendor/RH56F1/RH56F1_L/meshes/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; visual mesh filename=file:///home/user/rl_ws/urdf/vendor/RH56F1/RH56F1_L/meshes/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
- link l_hl_index_tip: geometry collision mesh filename=file:///home/user/rl_ws/urdf/vendor/RH56F1/RH56F1_L/meshes/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; visual mesh filename=file:///home/user/rl_ws/urdf/vendor/RH56F1/RH56F1_L/meshes/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
- link l_hl_middle_1: geometry collision mesh filename=file:///home/user/rl_ws/urdf/vendor/RH56F1/RH56F1_L/meshes/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; visual mesh filename=file:///home/user/rl_ws/urdf/vendor/RH56F1/RH56F1_L/meshes/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
- link l_hl_middle_2: geometry collision mesh filename=file:///home/user/rl_ws/urdf/vendor/RH56F1/RH56F1_L/meshes/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; visual mesh filename=file:///home/user/rl_ws/urdf/vendor/RH56F1/RH56F1_L/meshes/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
- link l_hl_middle_sensor: geometry collision mesh filename=file:///home/user/rl_ws/urdf/vendor/RH56F1/RH56F1_L/meshes/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; visual mesh filename=file:///home/user/rl_ws/urdf/vendor/RH56F1/RH56F1_L/meshes/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
- link l_hl_middle_tip: geometry collision mesh filename=file:///home/user/rl_ws/urdf/vendor/RH56F1/RH56F1_L/meshes/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; visual mesh filename=file:///home/user/rl_ws/urdf/vendor/RH56F1/RH56F1_L/meshes/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
- link l_hl_palm_1: geometry collision mesh filename=file:///home/user/rl_ws/urdf/vendor/RH56F1/RH56F1_L/meshes/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; visual mesh filename=file:///home/user/rl_ws/urdf/vendor/RH56F1/RH56F1_L/meshes/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
- link l_hl_pinky_1: geometry collision mesh filename=file:///home/user/rl_ws/urdf/vendor/RH56F1/RH56F1_L/meshes/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; visual mesh filename=file:///home/user/rl_ws/urdf/vendor/RH56F1/RH56F1_L/meshes/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
- link l_hl_pinky_2: geometry collision mesh filename=file:///home/user/rl_ws/urdf/vendor/RH56F1/RH56F1_L/meshes/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; visual mesh filename=file:///home/user/rl_ws/urdf/vendor/RH56F1/RH56F1_L/meshes/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
- link l_hl_pinky_sensor: geometry collision mesh filename=file:///home/user/rl_ws/urdf/vendor/RH56F1/RH56F1_L/meshes/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; visual mesh filename=file:///home/user/rl_ws/urdf/vendor/RH56F1/RH56F1_L/meshes/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
- link l_hl_pinky_tip: geometry collision mesh filename=file:///home/user/rl_ws/urdf/vendor/RH56F1/RH56F1_L/meshes/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; visual mesh filename=file:///home/user/rl_ws/urdf/vendor/RH56F1/RH56F1_L/meshes/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
- link l_hl_ring_1: geometry collision mesh filename=file:///home/user/rl_ws/urdf/vendor/RH56F1/RH56F1_L/meshes/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; visual mesh filename=file:///home/user/rl_ws/urdf/vendor/RH56F1/RH56F1_L/meshes/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
- link l_hl_ring_2: geometry collision mesh filename=file:///home/user/rl_ws/urdf/vendor/RH56F1/RH56F1_L/meshes/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; visual mesh filename=file:///home/user/rl_ws/urdf/vendor/RH56F1/RH56F1_L/meshes/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
- link l_hl_ring_sensor: geometry collision mesh filename=file:///home/user/rl_ws/urdf/vendor/RH56F1/RH56F1_L/meshes/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; visual mesh filename=file:///home/user/rl_ws/urdf/vendor/RH56F1/RH56F1_L/meshes/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
- link l_hl_ring_tip: geometry collision mesh filename=file:///home/user/rl_ws/urdf/vendor/RH56F1/RH56F1_L/meshes/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; visual mesh filename=file:///home/user/rl_ws/urdf/vendor/RH56F1/RH56F1_L/meshes/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
- link l_hl_thumb_1: geometry collision mesh filename=file:///home/user/rl_ws/urdf/vendor/RH56F1/RH56F1_L/meshes/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; visual mesh filename=file:///home/user/rl_ws/urdf/vendor/RH56F1/RH56F1_L/meshes/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
- link l_hl_thumb_2: geometry collision mesh filename=file:///home/user/rl_ws/urdf/vendor/RH56F1/RH56F1_L/meshes/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; visual mesh filename=file:///home/user/rl_ws/urdf/vendor/RH56F1/RH56F1_L/meshes/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
- link l_hl_thumb_3: geometry collision mesh filename=file:///home/user/rl_ws/urdf/vendor/RH56F1/RH56F1_L/meshes/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; visual mesh filename=file:///home/user/rl_ws/urdf/vendor/RH56F1/RH56F1_L/meshes/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
- link l_hl_thumb_4: geometry collision mesh filename=file:///home/user/rl_ws/urdf/vendor/RH56F1/RH56F1_L/meshes/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; visual mesh filename=file:///home/user/rl_ws/urdf/vendor/RH56F1/RH56F1_L/meshes/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
- link l_hl_thumb_sensor: geometry collision mesh filename=file:///home/user/rl_ws/urdf/vendor/RH56F1/RH56F1_L/meshes/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; visual mesh filename=file:///home/user/rl_ws/urdf/vendor/RH56F1/RH56F1_L/meshes/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
- link l_hl_thumb_tip: geometry collision mesh filename=file:///home/user/rl_ws/urdf/vendor/RH56F1/RH56F1_L/meshes/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; visual mesh filename=file:///home/user/rl_ws/urdf/vendor/RH56F1/RH56F1_L/meshes/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
- link r_hl_index_1: geometry collision mesh filename=file:///home/user/rl_ws/urdf/vendor/RH56F1/RH56F1_R/meshes/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; visual mesh filename=file:///home/user/rl_ws/urdf/vendor/RH56F1/RH56F1_R/meshes/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
- link r_hl_index_2: geometry collision mesh filename=file:///home/user/rl_ws/urdf/vendor/RH56F1/RH56F1_R/meshes/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; visual mesh filename=file:///home/user/rl_ws/urdf/vendor/RH56F1/RH56F1_R/meshes/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
- link r_hl_index_sensor: geometry collision mesh filename=file:///home/user/rl_ws/urdf/vendor/RH56F1/RH56F1_R/meshes/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; visual mesh filename=file:///home/user/rl_ws/urdf/vendor/RH56F1/RH56F1_R/meshes/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
- link r_hl_index_tip: geometry collision mesh filename=file:///home/user/rl_ws/urdf/vendor/RH56F1/RH56F1_R/meshes/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; visual mesh filename=file:///home/user/rl_ws/urdf/vendor/RH56F1/RH56F1_R/meshes/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
- link r_hl_middle_1: geometry collision mesh filename=file:///home/user/rl_ws/urdf/vendor/RH56F1/RH56F1_R/meshes/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; visual mesh filename=file:///home/user/rl_ws/urdf/vendor/RH56F1/RH56F1_R/meshes/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
- link r_hl_middle_2: geometry collision mesh filename=file:///home/user/rl_ws/urdf/vendor/RH56F1/RH56F1_R/meshes/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; visual mesh filename=file:///home/user/rl_ws/urdf/vendor/RH56F1/RH56F1_R/meshes/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
- link r_hl_middle_sensor: geometry collision mesh filename=file:///home/user/rl_ws/urdf/vendor/RH56F1/RH56F1_R/meshes/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; visual mesh filename=file:///home/user/rl_ws/urdf/vendor/RH56F1/RH56F1_R/meshes/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
- link r_hl_middle_tip: geometry collision mesh filename=file:///home/user/rl_ws/urdf/vendor/RH56F1/RH56F1_R/meshes/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; visual mesh filename=file:///home/user/rl_ws/urdf/vendor/RH56F1/RH56F1_R/meshes/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
- link r_hl_palm_1: geometry collision mesh filename=file:///home/user/rl_ws/urdf/vendor/RH56F1/RH56F1_R/meshes/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; visual mesh filename=file:///home/user/rl_ws/urdf/vendor/RH56F1/RH56F1_R/meshes/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
- link r_hl_pinky_1: geometry collision mesh filename=file:///home/user/rl_ws/urdf/vendor/RH56F1/RH56F1_R/meshes/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; visual mesh filename=file:///home/user/rl_ws/urdf/vendor/RH56F1/RH56F1_R/meshes/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
- link r_hl_pinky_2: geometry collision mesh filename=file:///home/user/rl_ws/urdf/vendor/RH56F1/RH56F1_R/meshes/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; visual mesh filename=file:///home/user/rl_ws/urdf/vendor/RH56F1/RH56F1_R/meshes/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
- link r_hl_pinky_sensor: geometry collision mesh filename=file:///home/user/rl_ws/urdf/vendor/RH56F1/RH56F1_R/meshes/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; visual mesh filename=file:///home/user/rl_ws/urdf/vendor/RH56F1/RH56F1_R/meshes/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
- link r_hl_pinky_tip: geometry collision mesh filename=file:///home/user/rl_ws/urdf/vendor/RH56F1/RH56F1_R/meshes/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; visual mesh filename=file:///home/user/rl_ws/urdf/vendor/RH56F1/RH56F1_R/meshes/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
- link r_hl_ring_1: geometry collision mesh filename=file:///home/user/rl_ws/urdf/vendor/RH56F1/RH56F1_R/meshes/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; visual mesh filename=file:///home/user/rl_ws/urdf/vendor/RH56F1/RH56F1_R/meshes/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
- link r_hl_ring_2: geometry collision mesh filename=file:///home/user/rl_ws/urdf/vendor/RH56F1/RH56F1_R/meshes/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; visual mesh filename=file:///home/user/rl_ws/urdf/vendor/RH56F1/RH56F1_R/meshes/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
- link r_hl_ring_sensor: geometry collision mesh filename=file:///home/user/rl_ws/urdf/vendor/RH56F1/RH56F1_R/meshes/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; visual mesh filename=file:///home/user/rl_ws/urdf/vendor/RH56F1/RH56F1_R/meshes/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
- link r_hl_ring_tip: geometry collision mesh filename=file:///home/user/rl_ws/urdf/vendor/RH56F1/RH56F1_R/meshes/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; visual mesh filename=file:///home/user/rl_ws/urdf/vendor/RH56F1/RH56F1_R/meshes/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
- link r_hl_thumb_1: geometry collision mesh filename=file:///home/user/rl_ws/urdf/vendor/RH56F1/RH56F1_R/meshes/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; visual mesh filename=file:///home/user/rl_ws/urdf/vendor/RH56F1/RH56F1_R/meshes/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
- link r_hl_thumb_2: geometry collision mesh filename=file:///home/user/rl_ws/urdf/vendor/RH56F1/RH56F1_R/meshes/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; visual mesh filename=file:///home/user/rl_ws/urdf/vendor/RH56F1/RH56F1_R/meshes/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
- link r_hl_thumb_3: geometry collision mesh filename=file:///home/user/rl_ws/urdf/vendor/RH56F1/RH56F1_R/meshes/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; visual mesh filename=file:///home/user/rl_ws/urdf/vendor/RH56F1/RH56F1_R/meshes/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
- link r_hl_thumb_4: geometry collision mesh filename=file:///home/user/rl_ws/urdf/vendor/RH56F1/RH56F1_R/meshes/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; visual mesh filename=file:///home/user/rl_ws/urdf/vendor/RH56F1/RH56F1_R/meshes/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
- link r_hl_thumb_sensor: geometry collision mesh filename=file:///home/user/rl_ws/urdf/vendor/RH56F1/RH56F1_R/meshes/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; visual mesh filename=file:///home/user/rl_ws/urdf/vendor/RH56F1/RH56F1_R/meshes/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
- link r_hl_thumb_tip: geometry collision mesh filename=file:///home/user/rl_ws/urdf/vendor/RH56F1/RH56F1_R/meshes/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; visual mesh filename=file:///home/user/rl_ws/urdf/vendor/RH56F1/RH56F1_R/meshes/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

Commit message: fix(assets,pour_fabric_mimic): RH56F1 손끝 collider 를 _sensor 하나로 — 벤더 STL 3중 사본 제거 + palm_1/2 decomposition
- 벤더 STL 의 {f}_2·{f}_force_sensor·{f}_tip(엄지 thumb_4·sensor·tip)은 같은 입체(면·부피·관성 동일)라
  한 마디에 강체 셋이 겹쳐 자기충돌 ON 117~558 N 상시접촉·접촉 임의 분할. collider 는 _sensor 에만(사용자 결정),
  _2·_tip 은 질량·visual·프레임 유지(유령 아님 — _sensor 가 같은 입체를 차지하고 fixed 로 _2 에 힘 전달).
- palm_1·palm_2 hull 이 palm_sensor 패드 면을 1~5 mm 덮어 컵이 센서보다 먼저 닿음 → 두 껍질만 convexDecomposition.
- 자산: 76 강체 · convexHull 51 + convexDecomposition 4 · 필터 50쌍 · mimic 12(nf 500).
- pour_fabric_mimic 프로필 finger_sensor_bodies=(_1, _sensor)(엄지 thumb_3, thumb_sensor), side_rig 2원소=원위/팁=센서.
  촉각 obs·접촉 동결·손가락 접촉력이 _sensor 를 읽는다 → obs 의미 변경, 재학습 필요. 테스트: 접촉 링크 collider 보유·사본 무 collider.
- 프로브: --obstacle_mm(palm_sensor 앞 키네마틱 큐브)·--contact_partners 절대경로.

Co-Authored-By: Claude Opus 5 <noreply@anthropic.com>
Claude-Session: https://claude.ai/code/session_016RobHoZyV19R1xziMustBN

File: assets/robot/openarm_rh56f1_bi_rl/openarm_rh56f1_bi_rl.urdf (robot description, URDF)
Before this commit: robot openarm_rh56f1_bi_rl, 76 links, 75 joints
Links:
- link l_hl_index_2: geometry visual mesh filename=file:///home/user/rl_ws/urdf/vendor/RH56F1/RH56F1_L/meshes/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
- link l_hl_index_tip: geometry visual mesh filename=file:///home/user/rl_ws/urdf/vendor/RH56F1/RH56F1_L/meshes/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
- link l_hl_middle_2: geometry visual mesh filename=file:///home/user/rl_ws/urdf/vendor/RH56F1/RH56F1_L/meshes/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
- link l_hl_middle_tip: geometry visual mesh filename=file:///home/user/rl_ws/urdf/vendor/RH56F1/RH56F1_L/meshes/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
- link l_hl_pinky_2: geometry visual mesh filename=file:///home/user/rl_ws/urdf/vendor/RH56F1/RH56F1_L/meshes/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
- link l_hl_pinky_tip: geometry visual mesh filename=file:///home/user/rl_ws/urdf/vendor/RH56F1/RH56F1_L/meshes/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
- link l_hl_ring_2: geometry visual mesh filename=file:///home/user/rl_ws/urdf/vendor/RH56F1/RH56F1_L/meshes/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
- link l_hl_ring_tip: geometry visual mesh filename=file:///home/user/rl_ws/urdf/vendor/RH56F1/RH56F1_L/meshes/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
- link l_hl_thumb_4: geometry visual mesh filename=file:///home/user/rl_ws/urdf/vendor/RH56F1/RH56F1_L/meshes/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
- link l_hl_thumb_tip: geometry visual mesh filename=file:///home/user/rl_ws/urdf/vendor/RH56F1/RH56F1_L/meshes/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
- link r_hl_index_2: geometry visual mesh filename=file:///home/user/rl_ws/urdf/vendor/RH56F1/RH56F1_R/meshes/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
- link r_hl_index_tip: geometry visual mesh filename=file:///home/user/rl_ws/urdf/vendor/RH56F1/RH56F1_R/meshes/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
- link r_hl_middle_2: geometry visual mesh filename=file:///home/user/rl_ws/urdf/vendor/RH56F1/RH56F1_R/meshes/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
- link r_hl_middle_tip: geometry visual mesh filename=file:///home/user/rl_ws/urdf/vendor/RH56F1/RH56F1_R/meshes/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
- link r_hl_pinky_2: geometry visual mesh filename=file:///home/user/rl_ws/urdf/vendor/RH56F1/RH56F1_R/meshes/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
- link r_hl_pinky_tip: geometry visual mesh filename=file:///home/user/rl_ws/urdf/vendor/RH56F1/RH56F1_R/meshes/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
- link r_hl_ring_2: geometry visual mesh filename=file:///home/user/rl_ws/urdf/vendor/RH56F1/RH56F1_R/meshes/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
- link r_hl_ring_tip: geometry visual mesh filename=file:///home/user/rl_ws/urdf/vendor/RH56F1/RH56F1_R/meshes/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
- link r_hl_thumb_4: geometry visual mesh filename=file:///home/user/rl_ws/urdf/vendor/RH56F1/RH56F1_R/meshes/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
- link r_hl_thumb_tip: geometry visual mesh filename=file:///home/user/rl_ws/urdf/vendor/RH56F1/RH56F1_R/meshes/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
